File: SUMEC V7/SUMEC V7.kicad_pcb (KiCad board)
At the start: 2 copper layers, 90.5 x 61 mm, 31 parts, among them IC1 XT30U-M, J1 Conn_01x04_Male, J2 Conn_01x04_Male, J3 Conn_01x03_Male, J4 Conn_01x05_Male, J5 Conn_01x03_Male, U1 QRE1113, U11 LD1086V33-DG, U12 LM7805_TO220, U2 QRE1113, U3 QRE1113, U4 QRE1113, U5 TSOP382xx, U6 Pico, U7 ROB-14450

Commit message: Update SUMEC V7.kicad_pcb
Parts:
- H3: footprint MountingHole:MountingHole_2.2mm_M2_ISO7380 -> MountingHole:MountingHole_3.2mm_M3
- moved R7 2.30 mm to (90.2, 38.1), turned to -90 degrees
Routing:
- net Net-(U4-A): track 0.00 -> 2.14 mm
- net QRE1113 A: track 24.6 -> 23.4 mm
- net +12V: track 80.9 -> 81.5 mm
