File: SUMEC V7/SUMEC V7.kicad_sch (KiCad schematic)
At the start: 34 parts, among them IC1 XT30U-M, J1 Conn_01x04_Male, J2 Conn_01x04_Male, J3 Conn_01x03_Male, J4 Conn_01x05_Male, J5 Conn_01x03_Male, U1 QRE1113, U10 VL53L0X, U11 LD1086V33-DG, U12 LM7805_TO220, U2 QRE1113, U3 QRE1113, U4 QRE1113, U5 TSOP382xx, U6 Pico, U7 ROB-14450, U8 VL53L0X, U9 VL53L0X

Commit message: Update SUMEC V7.kicad_sch
Parts:
- H1: value MountingHole M2 -> MountingHole; footprint MountingHole:MountingHole_2.2mm_M2_ISO14580 -> MountingHole:MountingHole_3.2mm_M3_DIN965
- H3: footprint MountingHole:MountingHole_2.2mm_M2_ISO7380 -> MountingHole:MountingHole_3.2mm_M3
