File: SUMEC GITHUB/SUMEC GIT.kicad_sch (KiCad schematic)
At the start: 35 parts, among them IC1 XT30U-M, J1 Conn_01x05_Pin, J2 Conn_01x05_Pin, J3 Conn_01x05_Pin, J4 Conn_01x05_Male, J5 Conn_01x03_Male, J6 Conn_01x03_Male, U1 QRE1113, U10 VL53L0X, U11 LD1086V33-DG, U12 LM7805_TO220, U2 QRE1113, U3 QRE1113, U4 QRE1113, U5 TSOP382xx, U6 Pico, U7 ROB-14450, U8 VL53L0X, U9 VL53L0X

Commit message: V8.1
Connections:
- net X-SHUT 1: now reaches U6.5 (GPIO3)
- net X-SHUT 1: now also J1.3 (Pin_3)
- removed net X-SHUT: J1.3 (Pin_3), J2.3 (Pin_3), J3.3 (Pin_3), U6.15 (GPIO11), U6.16 (GPIO12), U6.17 (GPIO13)
- new net X-SHUT 2: J2.3 (Pin_3), U6.16 (GPIO12)
- new net X-SHUT 3: J3.3 (Pin_3), U6.17 (GPIO13)
Changed lines of the file:
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@@
   (no_connect (at 262.89 182.88))
   (no_connect (at 92.71 217.17))
-  (no_connect (at 220.98 180.34))
   (no_connect (at 100.33 217.17))
   (no_connect (at 110.49 217.17))
@@
   (no_connect (at 220.98 193.04))
   (no_connect (at 158.75 217.17))
+  (no_connect (at 222.25 205.74))
   (no_connect (at 262.89 177.8))
   (polyline (pts (xy 345.44 228.6) (xy 358.14 228.6))
@@
     )
   )
-  (global_label "X-SHUT" (shape input) (at 187.96 77.47 0) (fields_autoplaced)
+  (global_label "X-SHUT 3" (shape input) (at 187.96 77.47 0) (fields_autoplaced)
     (effects (font (size 1 1)) (justify left))
-    (property "Intersheetrefs" "${INTERSHEET_REFS}" (at 196.2479 77.47 0)
+    (property "Intersheetrefs" "${INTERSHEET_REFS}" (at 197.8003 77.47 0)
       (effects (font (size 1.27 1.27)) (justify left) hide)
     )
@@
     )
   )
+  (global_label "X-SHUT 1" (shape input) (at 220.98 180.34 180) (fields_autoplaced)
+    (effects (font (size 1 1)) (justify right))
+    (property "Intersheetrefs" "${INTERSHEET_REFS}" (at 211.1397 180.34 0)
+      (effects (font (size 1.27 1.27)) (justify right) hide)
+    )
+  )
+  (global_label "X-SHUT 2" (shape input) (at 222.25 208.28 180) (fields_autoplaced)
+    (effects (font (size 1 1)) (justify right))
+    (property "Intersheetrefs" "${INTERSHEET_REFS}" (at 212.4097 208.28 0)
+      (effects (font (size 1.27 1.27)) (justify right) hide)
+    )
+  )
   (global_label "MOTOR 2 -" (shape input) (at 106.68 73.66 0) (fields_autoplaced)
     (effects (font (size 1.27 1.27)) (justify left))
@@
     (effects (font (size 1.27 1.27)) (justify left))
     (property "Intersheetrefs" "${INTERSHEET_REFS}" (at 145.6812 160.0994 0)
-      (effects (font (size 1.27 1.27)) (justify left) hide)
-    )
-  )
-  (global_label "X-SHUT" (shape input) (at 138.43 77.47 0) (fields_autoplaced)
-    (effects (font (size 1 1)) (justify left))
-    (property "Intersheetrefs" "${INTERSHEET_REFS}" (at 146.7179 77.47 0)
       (effects (font (size 1.27 1.27)) (justify left) hide)
     )
@@
     )
   )
+  (global_label "X-SHUT 1" (shape input) (at 138.43 77.47 0) (fields_autoplaced)
+    (effects (font (size 1 1)) (justify left))
+    (property "Intersheetrefs" "${INTERSHEET_REFS}" (at 148.2703 77.47 0)
+      (effects (font (size 1.27 1.27)) (justify left) hide)
+    )
+  )
   (global_label "QRE1113 D" (shape input) (at 318.77 222.25 0) (fields_autoplaced)
     (effects (font (size 1.27 1.27)) (justify left))
@@
     )
   )
-  (global_label "X-SHUT" (shape input) (at 222.25 205.74 180) (fields_autoplaced)
+  (global_label "X-SHUT 3" (shape input) (at 222.25 210.82 180) (fields_autoplaced)
     (effects (font (size 1 1)) (justify right))
-    (property "Intersheetrefs" "${INTERSHEET_REFS}" (at 213.9621 205.74 0)
+    (property "Intersheetrefs" "${INTERSHEET_REFS}" (at 212.4097 210.82 0)
       (effects (font (size 1.27 1.27)) (justify right) hide)
     )
@@
     )
   )
-  (global_label "X-SHUT" (shape input) (at 165.1 77.47 0) (fields_autoplaced)
+  (global_label "X-SHUT 2" (shape input) (at 165.1 77.47 0) (fields_autoplaced)
     (effects (font (size 1 1)) (justify left))
-    (property "Intersheetrefs" "${INTERSHEET_REFS}" (at 173.3879 77.47 0)
+    (property "Intersheetrefs" "${INTERSHEET_REFS}" (at 174.9403 77.47 0)
       (effects (font (size 1.27 1.27)) (justify left) hide)
     )
@@
     )
   )
-  (global_label "X-SHUT" (shape input) (at 222.25 210.82 180) (fields_autoplaced)
-    (effects (font (size 1 1)) (justify right))
-    (property "Intersheetrefs" "${INTERSHEET_REFS}" (at 213.9621 210.82 0)
-      (effects (font (size 1.27 1.27)) (justify right) hide)
-    )
-  )
   (global_label "BI1" (shape input) (at 223.52 124.46 180) (fields_autoplaced)
     (effects (font (size 1.27 1.27)) (justify right))
@@
       (effects (font (size 1.27 1.27)) (justify right) hide)
     )
-  )
-  (global_label "X-SHUT" (shape input) (at 222.25 208.28 180) (fields_autoplaced)
-    (effects (font (size 1 1)) (justify right))
-    (property "Intersheetrefs" "${INTERSHEET_REFS}" (at 213.9621 208.28 0)
-      (effects (font (size 1.27 1.27)) (justify right) hide)
-    )

Commit message: Update SUMEC GIT.kicad_sch
Parts:
- J5: footprint Connector_PinSocket_2.54mm:PinSocket_1x02_P2.54mm_Vertical -> Connector_PinSocket_2.54mm:PinSocket_1x03_P2.54mm_Vertical
Changed lines of the file:
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@@
       (effects (font (size 1.27 1.27)))
     )
-    (property "Footprint" "Connector_PinSocket_2.54mm:PinSocket_1x02_P2.54mm_Vertical" (at 77.47 125.73 0)
+    (property "Footprint" "Connector_PinSocket_2.54mm:PinSocket_1x03_P2.54mm_Vertical" (at 77.47 125.73 0)
       (effects (font (size 1.27 1.27)) hide)
     )

Commit message: V9
Connections:
- net +12V: now also J5.1 (Pin_1); no longer J5.2 (Pin_2)
- net AI1: now also U6.11 (GPIO8); no longer U6.26 (GPIO20)
- net GND: now also J5.2 (Pin_2), J6.2 (Pin_2); no longer J5.1 (Pin_1), J6.1 (Pin_1)
- net IR MODULE: now also J6.1 (Pin_1), U6.19 (GPIO14); no longer J6.2 (Pin_2), U6.11 (GPIO8)
