File: SUMEC GITHUB/SUMEC GIT.kicad_pcb (KiCad board)
At the start: 2 copper layers, 90.5 x 100.2 mm, 31 parts, among them IC1 XT30U-M, J1 Conn_01x05_Pin, J2 Conn_01x05_Pin, J3 Conn_01x05_Pin, J4 Conn_01x05_Male, J5 Conn_01x03_Male, J6 Conn_01x03_Male, U1 QRE1113, U11 LD1086V33-DG, U12 LM7805_TO220, U2 QRE1113, U3 QRE1113, U4 QRE1113, U6 Pico, U7 ROB-14450

Commit message: V8.1
Parts:
- J5: footprint Connector_PinSocket_2.54mm:PinSocket_1x02_P2.54mm_Vertical -> Connector_PinSocket_2.54mm:PinSocket_1x03_P2.54mm_Vertical
- moved C3 18.6 mm to (111.5, 86.6), turned to 180 degrees
- moved U11 10.1 mm to (115.7, 86.5), turned to 0 degrees
- moved C4 8.48 mm to (125.0, 86.6), turned to 0 degrees
- moved J5 1.28 mm to (123.2, 54.0)
Connections:
- J1 pad 3: X-SHUT -> X-SHUT 1
- J2 pad 3: X-SHUT -> X-SHUT 2
- J3 pad 3: X-SHUT -> X-SHUT 3
- U6 pad 15: X-SHUT -> unconnected-(U6-GPIO11-Pad15)
- U6 pad 16: X-SHUT -> X-SHUT 2
- U6 pad 17: X-SHUT -> X-SHUT 3
- U6 pad 5: unconnected-(U6-GPIO3-Pad5) -> X-SHUT 1
Routing:
- net X-SHUT: track 70.7 -> 0.00 mm, vias 2 -> 0
- net X-SHUT 3: track 0.00 -> 44.4 mm
- net X-SHUT 1: track 0.00 -> 14.0 mm
- net X-SHUT 2: track 0.00 -> 13.9 mm
- net +3V3: track 224.5 -> 232.6 mm
- net +12V: track 82.4 -> 81.5 mm

Commit message: V8.2
Parts:
- moved J5 2.84 mm to (125.5, 55.8)
- moved IC1 1.77 mm to (92.8, 55.8)
Connections:
- J5 pad 1: GND -> +12V
Routing:
- net +5V: track 31.7 -> 95.2 mm
- net +12V: track 81.5 -> 50.9 mm
Changed lines of the file:
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@@
     (pad_to_mask_clearance 0)
     (pcbplotparams
-      (layerselection 0x00010fc_ffffffff)
-      (plot_on_all_layers_selection 0x0000000_00000000)
+      (layerselection 0x0000000_7fffffff)
+      (plot_on_all_layers_selection 0x0000000_00000001)
       (disableapertmacros false)
       (usegerberextensions false)
@@
       (dxfimperialunits true)
       (dxfusepcbnewfont true)
-      (psnegative false)
+      (psnegative true)
       (psa4output false)
       (plotreference true)
@@
       (sketchpadsonfab false)
       (subtractmaskfromsilk false)
-      (outputformat 1)
+      (outputformat 4)
       (mirror false)
-      (drillshape 1)
+      (drillshape 2)
       (scaleselection 1)
       (outputdirectory "")
@@
   )
   (footprint "Connector_PinSocket_2.54mm:PinSocket_1x03_P2.54mm_Vertical" (layer "F.Cu")
-    (at 123.25 54.025 -90)
+    (at 125.5 55.75 -90)
     (descr "Through hole straight socket strip, 1x03, 2.54mm pitch, single row (from Kicad 4.0.7), script generated")
     (tags "Through hole socket strip THT 1x03 2.54mm single row")
@@
       (stroke (width 0.1) (type solid)) (layer "F.Fab"))
     (pad "1" thru_hole rect (at 0 0 270) (size 1.7 1.7) (drill 1) (layers "*.Cu" "*.Mask")
-      (net 1 "GND") (pinfunction "Pin_1") (pintype "passive"))
+      (net 16 "+12V") (pinfunction "Pin_1") (pintype "passive"))
     (pad "2" thru_hole oval (at 0 2.54 270) (size 1.7 1.7) (drill 1) (layers "*.Cu" "*.Mask")
       (net 16 "+12V") (pinfunction "Pin_2") (pintype "passive"))
@@
   )
   (footprint "Connector_AMASS:AMASS_XT30U-M_1x02_P5.0mm_Vertical" (layer "F.Cu")
-    (at 92.5 54)
+    (at 92.75 55.75)
     (descr "Connector XT30 Vertical Cable Male, https://www.tme.eu/en/Document/3cbfa5cfa544d79584972dd5234a409e/XT30U%20SPEC.pdf")
     (tags "RC Connector XT30")
@@
   (segment (start 85.71 55.96) (end 58.25 55.96) (width 0.5) (layer "F.Cu") (net 5))
   (via (at 85.75 56) (size 2) (drill 1) (layers "F.Cu" "B.Cu") (free) (net 5))
+  (segment (start 85.75 56) (end 89.25 52.5) (width 0.5) (layer "B.Cu") (net 5))
+  (segment (start 131.5 52.5) (end 132.75 53.75) (width 0.5) (layer "B.Cu") (net 5))
+  (segment (start 89.25 52.5) (end 131.5 52.5) (width 0.5) (layer "B.Cu") (net 5))
+  (segment (start 131.5 66.25) (end 130 66.25) (width 0.5) (layer "B.Cu") (net 5))
+  (segment (start 132.75 53.75) (end 132.75 65) (width 0.5) (layer "B.Cu") (net 5))
   (segment (start 130 66.25) (end 130 70.405) (width 0.5) (layer "B.Cu") (net 5))
+  (segment (start 132.75 65) (end 131.5 66.25) (width 0.5) (layer "B.Cu") (net 5))
   (segment (start 130 70.405) (end 129.945 70.46) (width 0.5) (layer "B.Cu") (net 5))
   (segment (start 139 93.25) (end 140.4 91.85) (width 0.5) (layer "B.Cu") (net 6))
@@
   (segment (start 130 88.75) (end 130 79.75) (width 0.5) (layer "B.Cu") (net 7))
   (segment (start 142.5 83.5) (end 142.5 81.5) (width 0.5) (layer "B.Cu") (net 7))
-  (segment (start 111.4 51.4) (end 111.5 51.5) (width 0.25) (layer "B.Cu") (net 7))
+  (segment (start 142.5 53.5) (end 142.5 81.5) (width 0.5) (layer "B.Cu") (net 7))
+  (segment (start 105.25 45.5) (end 88.245 45.5) (width 0.5) (layer "B.Cu") (net 7))
   (segment (start 123.25 88.75) (end 123.25 91.75) (width 0.5) (layer "B.Cu") (net 7))
-  (segment (start 111.5 45.505) (end 111.5 51.5) (width 0.5) (layer "B.Cu") (net 7))
   (segment (start 126.85 76.6) (end 124.62 76.6) (width 0.5) (layer "B.Cu") (net 7))
+  (segment (start 111.5 51.25) (end 111 51.25) (width 0.5) (layer "B.Cu") (net 7))
+  (segment (start 111.5 45.505) (end 111.5 51.25) (width 0.5) (layer "B.Cu") (net 7))
   (segment (start 96.17 91.75) (end 96.17 88.92) (width 0.5) (layer "B.Cu") (net 7))
+  (segment (start 111.495 45.5) (end 111.5 45.505) (width 0.5) (layer "B.Cu") (net 7))
   (segment (start 118.25 87.345) (end 118.25 86.5) (width 0.5) (layer "B.Cu") (net 7))
   (segment (start 139 83.5) (end 142.5 83.5) (width 0.5) (layer "B.Cu") (net 7))
@@
   (segment (start 116.925 85.175) (end 118.25 86.5) (width 0.25) (layer "B.Cu") (net 7))
   (segment (start 128.25 88.75) (end 130 88.75) (width 0.5) (layer "B.Cu") (net 7))
-  (segment (start 139.75 51.5) (end 142.5 54.25) (width 0.5) (layer "B.Cu") (net 7))
+  (segment (start 111.5 51.25) (end 140.25 51.25) (width 0.5) (layer "B.Cu") (net 7))
   (segment (start 118.25 86.5) (end 118.25 88.75) (width 0.25) (layer "B.Cu") (net 7))
   (segment (start 68.5 88.75) (end 83.5 88.75) (width 0.5) (layer "B.Cu") (net 7))
   (segment (start 123.25 88.75) (end 142.5 88.75) (width 0.5) (layer "B.Cu") (net 7))
   (segment (start 83.5 88.75) (end 96 88.75) (width 0.5) (layer "B.Cu") (net 7))
-  (segment (start 111.5 51.5) (end 139.75 51.5) (width 0.5) (layer "B.Cu") (net 7))
+  (segment (start 140.25 51.25) (end 142.5 53.5) (width 0.5) (layer "B.Cu") (net 7))
   (segment (start 63.505 88.75) (end 60.5 91.755) (width 0.5) (layer "B.Cu") (net 7))
-  (segment (start 111.495 45.5) (end 111.5 45.505) (width 0.5) (layer "B.Cu") (net 7))
   (segment (start 111.472599 86.555) (end 112.852599 85.175) (width 0.25) (layer "B.Cu") (net 7))
   (segment (start 142.5 88.75) (end 142.5 91.505) (width 0.5) (layer "B.Cu") (net 7))
   (segment (start 123.29 88.71) (end 123.25 88.75) (width 0.5) (layer "B.Cu") (net 7))
-  (segment (start 111.5 51.5) (end 111.25 51.5) (width 0.5) (layer "B.Cu") (net 7))
   (segment (start 83.54 86.5) (end 83.54 88.71) (width 0.5) (layer "B.Cu") (net 7))
   (segment (start 96.17 88.92) (end 96 88.75) (width 0.5) (layer "B.Cu") (net 7))
@@
   (segment (start 112.852599 85.175) (end 116.925 85.175) (width 0.25) (layer "B.Cu") (net 7))
   (segment (start 68.42 91.75) (end 68.42 88.83) (width 0.5) (layer "B.Cu") (net 7))
-  (segment (start 105.25 45.5) (end 88.245 45.5) (width 0.5) (layer "B.Cu") (net 7))
+  (segment (start 111 51.25) (end 105.25 45.5) (width 0.5) (layer "B.Cu") (net 7))
   (segment (start 118.25 88.75) (end 123.25 88.75) (width 0.5) (layer "B.Cu") (net 7))
   (segment (start 63.505 88.75) (end 68.5 88.75) (width 0.5) (layer "B.Cu") (net 7))
-  (segment (start 142.5 54.25) (end 142.5 81.5) (width 0.5) (layer "B.Cu") (net 7))
   (segment (start 130 79.75) (end 126.85 76.6) (width 0.5) (layer "B.Cu") (net 7))
-  (segment (start 111.25 51.5) (end 105.25 45.5) (width 0.5) (layer "B.Cu") (net 7))
   (segment (start 83.54 88.71) (end 83.5 88.75) (width 0.5) (layer "B.Cu") (net 7))
   (segment (start 68.42 88.83) (end 68.5 88.75) (width 0.5) (layer "B.Cu") (net 7))
@@
   (segment (start 88.25 37.75) (end 89.9 37.75) (width 0.5) (layer "F.Cu") (net 9))
   (segment (start 89.9 37.75) (end 90.25 38.1) (width 0.5) (layer "F.Cu") (net 9))
-  (segment (start 120.75 86.46) (end 120.79 86.5) (width 2) (layer "B.Cu") (net 16))
   (segment (start 120.79 86.5) (end 120.845 86.555) (width 2) (layer "B.Cu") (net 16))
-  (segment (start 97.5 54) (end 118.145 54) (width 2) (layer "B.Cu") (net 16))
   (segment (start 124.62 79.14) (end 121.36 79.14) (width 2) (layer "B.Cu") (net 16))
-  (segment (start 120.75 57.25) (end 120.75 86.46) (width 2) (layer "B.Cu") (net 16))
   (segment (start 120.845 86.555) (end 125 86.555) (width 2) (layer "B.Cu") (net 16))
-  (segment (start 129.945 57.1826) (end 120.8174 57.1826) (width 2) (layer "B.Cu") (net 16))
+  (segment (start 129.945 61.115) (end 130 61.17) (width 2) (layer "B.Cu") (net 16))
   (segment (start 129.945 57.1826) (end 129.945 61.115) (width 2) (layer "B.Cu") (net 16))
-  (segment (start 120.8174 57.1826) (end 120.75 57.25) (width 0.25) (layer "B.Cu") (net 16))
   (segment (start 120.79 79.71) (end 120.79 86.5) (width 2) (layer "B.Cu") (net 16))
-  (segment (start 120.71 54.025) (end 120.75 54.065) (width 2) (layer "B.Cu") (net 16))
-  (segment (start 129.945 61.115) (end 130 61.17) (width 2) (layer "B.Cu") (net 16))
-  (segment (start 120.75 54.065) (end 120.75 57.25) (width 2) (layer "B.Cu") (net 16))
-  (segment (start 118.145 54) (end 118.17 54.025) (width 2) (layer "B.Cu") (net 16))
+  (segment (start 129.945 57.1826) (end 129.6276 57.5) (width 0.25) (layer "B.Cu") (net 16))
+  (segment (start 122.96 55.75) (end 122.96 56.96) (width 2) (layer "B.Cu") (net 16))
+  (segment (start 124.25 58.25) (end 129.445 58.25) (width 2) (layer "B.Cu") (net 16))
+  (segment (start 97.75 55.75) (end 120.42 55.75) (width 2) (layer "B.Cu") (net 16))
+  (segment (start 120.75 86.46) (end 120.79 86.5) (width 2) (layer "B.Cu") (net 16))
+  (segment (start 122.96 56.96) (end 124.25 58.25) (width 2) (layer "B.Cu") (net 16))
+  (segment (start 129.445 58.25) (end 129.695 58) (width 2) (layer "B.Cu") (net 16))
   (segment (start 121.36 79.14) (end 120.79 79.71) (width 2) (layer "B.Cu") (net 16))
   (segment (start 101.25 91.75) (end 101.25 93.425) (width 0.5) (layer "F.Cu") (net 21))

Commit message: V8.3
Routing:
- net +12V: track 50.9 -> 82.6 mm
Other:
- board size 90.5 x 100.2 mm -> 90.5 x 61 mm
- board text removed: "BATT."
- board text removed: "GND = ROZLITÁ ZÉM"
- board text removed: "VIA = DRÁTOVÁ PROPOJKA"
Changed lines of the file:
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@@
   (gr_line (start 83.75 50.5) (end 83.75 35.5)
     (stroke (width 0.1) (type solid)) (layer "Edge.Cuts"))
-  (gr_rect (start 76 103.75) (end 116 135.75)
-    (stroke (width 0.2) (type default)) (fill none) (layer "Edge.Cuts"))
-  (gr_text "VIA = DRÁTOVÁ PROPOJKA" (at 99.75 31.75) (layer "Dwgs.User")
-    (effects (font (size 1.5 1.5) (thickness 0.3)))
-  )
-  (gr_text "GND = ROZLITÁ ZÉM" (at 96 27) (layer "Dwgs.User")
-    (effects (font (size 1.5 1.5) (thickness 0.3)))
-  )
-  (gr_text "BATT." (at 92 107) (layer "Edge.Cuts")
-    (effects (font (size 1.5 1.5) (thickness 0.3) bold) (justify left bottom))
-  )
   (segment (start 58.25 58.5) (end 58.25 62.02) (width 0.5) (layer "F.Cu") (net 2))
   (segment (start 58.25 62.02) (end 58.16 62.11) (width 0.5) (layer "F.Cu") (net 2))
@@
   (segment (start 88.25 37.75) (end 89.9 37.75) (width 0.5) (layer "F.Cu") (net 9))
   (segment (start 89.9 37.75) (end 90.25 38.1) (width 0.5) (layer "F.Cu") (net 9))
+  (segment (start 122.96 55.75) (end 122.96 57.96) (width 2) (layer "B.Cu") (net 16))
   (segment (start 120.79 86.5) (end 120.845 86.555) (width 2) (layer "B.Cu") (net 16))
+  (segment (start 120.79 79.71) (end 120.79 86.5) (width 2) (layer "B.Cu") (net 16))
+  (segment (start 120.845 86.555) (end 125 86.555) (width 2) (layer "B.Cu") (net 16))
+  (segment (start 123.25 58.25) (end 124.25 58.25) (width 2) (layer "B.Cu") (net 16))
+  (segment (start 120.75 59.17) (end 121.67 58.25) (width 2) (layer "B.Cu") (net 16))
+  (segment (start 120.75 86.46) (end 120.75 59.17) (width 2) (layer "B.Cu") (net 16))
+  (segment (start 129.945 61.115) (end 130 61.17) (width 2) (layer "B.Cu") (net 16))
   (segment (start 124.62 79.14) (end 121.36 79.14) (width 2) (layer "B.Cu") (net 16))
-  (segment (start 120.845 86.555) (end 125 86.555) (width 2) (layer "B.Cu") (net 16))
-  (segment (start 129.945 61.115) (end 130 61.17) (width 2) (layer "B.Cu") (net 16))
   (segment (start 129.945 57.1826) (end 129.945 61.115) (width 2) (layer "B.Cu") (net 16))
-  (segment (start 120.79 79.71) (end 120.79 86.5) (width 2) (layer "B.Cu") (net 16))
   (segment (start 129.945 57.1826) (end 129.6276 57.5) (width 0.25) (layer "B.Cu") (net 16))
-  (segment (start 122.96 55.75) (end 122.96 56.96) (width 2) (layer "B.Cu") (net 16))
+  (segment (start 121.36 79.14) (end 120.79 79.71) (width 2) (layer "B.Cu") (net 16))
+  (segment (start 120.79 86.5) (end 120.75 86.46) (width 2) (layer "B.Cu") (net 16))
+  (segment (start 122.96 57.96) (end 123.25 58.25) (width 2) (layer "B.Cu") (net 16))
   (segment (start 124.25 58.25) (end 129.445 58.25) (width 2) (layer "B.Cu") (net 16))
   (segment (start 97.75 55.75) (end 120.42 55.75) (width 2) (layer "B.Cu") (net 16))
-  (segment (start 120.75 86.46) (end 120.79 86.5) (width 2) (layer "B.Cu") (net 16))
-  (segment (start 122.96 56.96) (end 124.25 58.25) (width 2) (layer "B.Cu") (net 16))
+  (segment (start 121.67 58.25) (end 124.25 58.25) (width 2) (layer "B.Cu") (net 16))
   (segment (start 129.445 58.25) (end 129.695 58) (width 2) (layer "B.Cu") (net 16))
-  (segment (start 121.36 79.14) (end 120.79 79.71) (width 2) (layer "B.Cu") (net 16))
   (segment (start 101.25 91.75) (end 101.25 93.425) (width 0.5) (layer "F.Cu") (net 21))
   (segment (start 73.5 91.75) (end 68.32 86.57) (width 0.5) (layer "F.Cu") (net 21))

Commit message: V9
Parts:
- moved J6 30.3 mm to (108.7, 84.4)
- moved C3 29.8 mm to (139.8, 77.3), turned to -90 degrees
- moved U11 27.5 mm to (139.7, 73.0), turned to 90 degrees
- moved C4 27.2 mm to (139.8, 63.8), turned to 90 degrees
- moved C2 6.83 mm to (129.9, 77.3)
- moved C1 6.83 mm to (129.9, 64.0)
- moved U12 6.83 mm to (130.0, 68.0)
- moved J1 5.53 mm to (65.3, 86.2)
- moved J3 5.51 mm to (120.4, 86.2)
- moved J2 5.50 mm to (93.7, 86.2)
- moved R9 4.75 mm to (139.0, 88.2)
- moved D1 1.25 mm to (58.2, 57.2)
Connections:
- J5 pad 2: +12V -> GND
- J6 pad 1: GND -> IR MODULE
- J6 pad 2: IR MODULE -> GND
- R9 pad 3: (no net) -> GND
- U6 pad 11: IR MODULE -> AI1
- U6 pad 19: unconnected-(U6-GPIO14-Pad19) -> IR MODULE
- U6 pad 26: AI1 -> unconnected-(U6-GPIO20-Pad26)
Routing:
- net +3V3: track 232.7 -> 251.9 mm
- net +5V: track 95.2 -> 76.7 mm, vias 1 -> 2
- net BI2: track 24.9 -> 9.97 mm
- net X-SHUT 3: track 44.4 -> 34.9 mm
- net PWMB: track 14.7 -> 6.24 mm
- net +12V: track 82.6 -> 74.8 mm
- net X-SHUT 1: track 14.0 -> 8.31 mm
- net X-SHUT 2: track 13.9 -> 8.59 mm
- net AI1: track 27.1 -> 31.4 mm
- net SCL: track 72.0 -> 68.4 mm
- net IR MODULE: track 6.62 -> 10.1 mm
- net SDA: track 71.9 -> 69.0 mm
- net Net-(D1-K): track 3.65 -> 4.90 mm

Commit message: V9.1
Routing:
- net +3V3: track 251.9 -> 254.6 mm
Changed lines of the file:
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@@
   (segment (start 140.4 91.5) (end 138.65 93.25) (width 0.5) (layer "F.Cu") (net 6))
   (segment (start 134.4 81.8) (end 134.4 88.6) (width 0.5) (layer "B.Cu") (net 7))
+  (segment (start 107.025 45.5) (end 88.245 45.5) (width 0.5) (layer "B.Cu") (net 7))
   (segment (start 123 81.8) (end 123.8 81.8) (width 0.5) (layer "B.Cu") (net 7))
   (segment (start 123.4 76.6) (end 123 77) (width 0.5) (layer "B.Cu") (net 7))
@@
   (segment (start 137.5 77) (end 137.5 74.25) (width 0.5) (layer "B.Cu") (net 7))
   (segment (start 139.695 70.5) (end 142.25 70.5) (width 0.5) (layer "B.Cu") (net 7))
-  (segment (start 109.75 51.25) (end 104 45.5) (width 0.5) (layer "B.Cu") (net 7))
+  (segment (start 108.15 51.25) (end 107.525 50.625) (width 0.5) (layer "B.Cu") (net 7))
   (segment (start 136.2 81.8) (end 137.5 80.5) (width 0.5) (layer "B.Cu") (net 7))
   (segment (start 111.5 45.505) (end 111.5 51.25) (width 0.5) (layer "B.Cu") (net 7))
@@
   (segment (start 123.8 81.8) (end 134.95 81.8) (width 0.5) (layer "B.Cu") (net 7))
   (segment (start 134.4 88.6) (end 133.6 89.4) (width 0.5) (layer "B.Cu") (net 7))
+  (segment (start 107.525 46) (end 107.025 45.5) (width 0.5) (layer "B.Cu") (net 7))
   (segment (start 142.5 88.75) (end 142.5 88.25) (width 0.5) (layer "B.Cu") (net 7))
   (segment (start 142.5 53.5) (end 142.5 70.25) (width 0.5) (layer "B.Cu") (net 7))
@@
   (segment (start 142.5 83.25) (end 142.5 81.5) (width 0.5) (layer "B.Cu") (net 7))
   (segment (start 111.5 51.25) (end 140.25 51.25) (width 0.5) (layer "B.Cu") (net 7))
+  (segment (start 111.5 51.25) (end 108.15 51.25) (width 0.5) (layer "B.Cu") (net 7))
   (segment (start 124.62 76.6) (end 123.4 76.6) (width 0.5) (layer "B.Cu") (net 7))
   (segment (start 138 70.5) (end 139.695 70.5) (width 0.5) (layer "B.Cu") (net 7))
@@
   (segment (start 142.5 88.75) (end 142.5 91.505) (width 0.5) (layer "B.Cu") (net 7))
   (segment (start 142.5 70.25) (end 142.5 81.5) (width 0.5) (layer "B.Cu") (net 7))
+  (segment (start 107.525 50.625) (end 107.525 46) (width 0.5) (layer "B.Cu") (net 7))
   (segment (start 142.5 81.5) (end 142.5 88.75) (width 0.5) (layer "B.Cu") (net 7))
   (segment (start 96.21 86.25) (end 96.21 89.39) (width 0.5) (layer "B.Cu") (net 7))
   (segment (start 68.65 89.4) (end 62.855 89.4) (width 0.5) (layer "B.Cu") (net 7))
-  (segment (start 104 45.5) (end 88.245 45.5) (width 0.5) (layer "B.Cu") (net 7))
   (segment (start 139.75 77.067401) (end 137.567401 77.067401) (width 0.5) (layer "B.Cu") (net 7))
-  (segment (start 111.5 51.25) (end 109.75 51.25) (width 0.5) (layer "B.Cu") (net 7))
   (segment (start 133.6 89.4) (end 68.65 89.4) (width 0.5) (layer "B.Cu") (net 7))
   (segment (start 142.25 70.5) (end 142.5 70.25) (width 0.25) (layer "B.Cu") (net 7))

Commit message: V9.2
Routing:
- net X-SHUT 2: track 8.59 -> 9.76 mm
- net QRE1113 C: track 47.9 -> 47.2 mm
