File: - PCB -/SENSORS.kicad_sch (KiCad schematic)
At the start: 17 parts, among them U11 VL53L0X, U13 VL53L0X, U14 VL53L0X, U5 QRE1113, U5 TSOP382xx, U6 QRE1113, U8 QRE1113, U9 QRE1113

Commit message: PCB - board update + footprint/3d models export
Parts:
- removed R14: 500, Potentiometer_THT:Potentiometer_ACP_CA9-V10_Vertical, symbol Device:R_Trim
- removed U6: QRE1113, OptoDevice:OnSemi_CASE100AQ, symbol Sensor_Proximity:QRE1113
- added U7: QRE1113, sumec_library:OnSemi_CASE100AQ - QRE1113, symbol Sensor_Proximity:QRE1113
- U6: renamed from U5; footprint OptoDevice:OnSemi_CASE100AQ -> sumec_library:OnSemi_CASE100AQ - QRE1113
- U8, U9: footprint OptoDevice:OnSemi_CASE100AQ -> sumec_library:OnSemi_CASE100AQ - QRE1113
- renumbered R9 to R?, R4 to R?, R13 to R?, R1 to R?, R10 to R?, R3 to R?, R2 to R?, R12 to R?, U11 to U2, U14 to U3, U13 to U4, U5 to U?
Connections:
- net TRIMMER INPUT is gone; now on net +3V3: R?.2, R?.2, R?.2, R?.2
- net GND: now also U7.2 (K), U7.4
- net QRE1113 B: now also U7.3
- net at R?.1: now also U7.1 (A)
Other:
- note added: "Miniature Reflective Object Sensor - QRE1113 IR reflectance sensor is comprised of two parts - an IR emitting LED and an IR sensitive phototransistor. Analog output A 100Ω resistor is placed in series with the LED to limit current. A 10kΩ resistor pulls the output pin high, but when the light from the LED is reflected back onto the phototransistor the output will begin to go lower. Operating volt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"
- note removed: "Miniature Reflective Object Sensor - QRE1113 IR reflectance sensor is comprised of two parts - an IR emitting LED and an IR sensitive phototransistor. Analog output Trimmer (500R) controls the IR LED intensity. A 100Ω resistor is placed in series with the LED to limit current. A 10kΩ resistor pulls the output pin high, but when the light from the LED is reflected back onto the phototransistor the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"
