File: - PCB -/_autosave-SENSORS.kicad_sch (KiCad schematic)
At the start: 16 parts, among them U2 VL53L0X, U3 VL53L0X, U4 VL53L0X, U6 QRE1113, U7 QRE1113, U8 QRE1113, U9 QRE1113

Commit message: PCB - Board update (?)
Parts:
- U?: footprint (none) -> Connector_PinSocket_2.54mm:PinSocket_1x03_P2.54mm_Vertical
Other:
- note removed: "NO FOOTPRINT ASSIGNED"
Changed lines of the file:
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@@
     (effects (font (size 1.5 1.5) italic) (justify left bottom))
-  )
-  (text "NO FOOTPRINT ASSIGNED" (at 132.08 193.04 0)
-    (effects (font (size 1.27 1.27)) (justify left bottom))
   )
   (text "SENZORY ČÁRÝ\n" (at 203.2 25.4 0)
@@
       (effects (font (size 1.27 1.27)) (justify right))
     )
-    (property "Footprint" "" (at 151.765 180.34 0)
-      (effects (font (size 1.27 1.27)) hide)
-    )
+    (property "Footprint" "Connector_PinSocket_2.54mm:PinSocket_1x03_P2.54mm_Vertical" (at 151.765 180.34 0)
+      (effects (font (size 1.27 1.27)) hide)
+    )
