File: - PCB -/_autosave-sumec.kicad_pcb (KiCad board)
At the start: 2 copper layers, 95 x 73 mm, 30 parts, among them IC1 XT30U-F, SW1 SW_SPDT, SW3 SW_Push, U1 ESP32-DEVKIT-V1, U10 LD1117AV33, U11 ROB-14450, U2 VL53L0X, U3 VL53L0X, U4 VL53L0X, U5 TSOP382xx, U6 QRE1113, U7 QRE1113, U8 QRE1113, U9 QRE1113

Commit message: PCB - Board update (?)
Routing:
- net QRE1113 C: track 65.7 -> 68.6 mm
- net QRE1113 B: track 116.6 -> 117.6 mm
- added copper zone on F.Cu, net GND
