File: - PCB -/SUMEC THT/sumec.kicad_pcb (KiCad board)
At the start: 2 copper layers, 95 x 73 mm, 34 parts, among them IC1 XT30U-F, J1 Conn_01x01_Pin, J2 Conn_01x01_Pin, J3 Conn_01x01_Pin, J4 Conn_01x01_Pin, SW1 SW_SPDT, SW3 SW_Push, U1 ESP32-DEVKIT-V1, U10 LD1117AV33, U11 ROB-14450, U2 VL53L0X, U3 VL53L0X, U4 VL53L0X, U5 TSOP382xx, U6 QRE1113, U7 QRE1113, U8 QRE1113, U9 QRE1113

Commit message: PCB Schematic SMD
Routing:
- removed copper zone on B.Cu, net GND
- removed copper zone on F.Cu, net GND
Changed lines of the file:
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@@
   (segment (start 109.49 71.72) (end 110.49 72.72) (width 0.508) (layer "B.Cu") (net 41))
   (segment (start 110.49 72.72) (end 110.49 76.454) (width 0.508) (layer "B.Cu") (net 41))
-  (zone (net 2) (net_name "GND") (layer "F.Cu") (hatch edge 0.5)
-    (connect_pads yes (clearance 0.5))
-    (min_thickness 0.25) (filled_areas_thickness no)
-    (fill yes (thermal_gap 0.5) (thermal_bridge_width 0.5) (smoothing fillet) (radius 1))
-    (polygon
-      (pts
-        (xy 189.4332 128.016)
-        (xy 86.9188 127.8636)
-        (xy 85.5472 56.5404)
-        (xy 106.2228 45.7708)
-        (xy 123.3636 44.444)
-        (xy 153.3636 44.444)
-        (xy 160.1216 47.244)
-        (xy 190.3476 48.8188)
-      )
-    )
-  )
   (zone (net 5) (net_name "12V IN") (layer "B.Cu") (hatch edge 0.5)
     (priority 2)
@@
       )
     )
-  )
-  (zone (net 2) (net_name "GND") (layer "B.Cu") (hatch edge 0.5)
-    (priority 1)
-    (connect_pads yes (clearance 0.5))
-    (min_thickness 0.25) (filled_areas_thickness no)
-    (fill yes (thermal_gap 0.5) (thermal_bridge_width 0.5) (smoothing fillet) (radius 1))
-    (polygon
-      (pts
-        (xy 80.264 40.132)
-        (xy 193.04 40.132)
-        (xy 192.024 132.588)
-        (xy 84.328 137.668)
-      )
-    )
