File: - PCB -/SUMEC SMD/_autosave-MCU.kicad_sch (KiCad schematic)
At the start: 15 parts, among them J2 USB3090-XX-X_REVE, SW2 SW_Push, SW4 SW_Push, U9 ESP32-S3-WROOM-2

Commit message: pcb updae
Connections:
- no-connect marks 2 -> 3
Other:
- note added: "GPIO0 has an internal pullup resistor, so if it is left unconnected then it will pull high."
Changed lines of the file:
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@@
   (no_connect (at 416.56 67.31))
   (no_connect (at 416.56 59.69))
+  (no_connect (at 273.05 167.64))
   (wire (pts (xy 426.72 74.93) (xy 457.2 74.93))
     (stroke (width 0) (type default))
@@
     (effects (font (size 2 2) bold) (justify left bottom))
   )
+  (text "GPIO0 has an internal pullup resistor, so if it is left unconnected then it will pull high."
+    (at 41.91 80.01 0)
+    (effects (font (size 1.27 1.27)) (justify left bottom))
+  )
   (text "Referenční board" (at 391.16 228.6 0)
