File: - PCB -/SUMEC SMD/MECHANICS.kicad_sch (KiCad schematic)
At the start: 9 parts, among them J1 Conn_01x01_Pin, SW1 SW_SPDT, SW3 SW_Push

Commit message: PCB SMD update
Other:
- title: SUMEC THT -> SUMEC SMD
Changed lines of the file:
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@@
   (paper "A4")
   (title_block
-    (title "SUMEC THT")
+    (title "SUMEC SMD")
     (company "SPŠ NA PROSEKU")
   )

Commit message: PCB Schematic SMD
Parts:
- SW3: footprint Button_Switch_THT:SW_PUSH_6mm -> Button_Switch_SMD:SW_SPST_B3U-1000P
Changed lines of the file:
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@@
       (effects (font (size 1.27 1.27)))
     )
-    (property "Footprint" "Button_Switch_THT:SW_PUSH_6mm" (at 92.71 125.73 0)
+    (property "Footprint" "Button_Switch_SMD:SW_SPST_B3U-1000P" (at 92.71 125.73 0)
       (effects (font (size 1.27 1.27)) hide)
     )

Commit message: PCB SMD update
Parts:
- removed J1 (x4): Conn_01x01_Pin, Connector_Wire:SolderWire-0.5sqmm_1x01_D0.9mm_OD2.3mm, symbol Connector:Conn_01x01_Pin
- added J1, J2, J3, J4: Conn_01x01_Pin, Connector_Wire:SolderWire-0.5sqmm_1x01_D0.9mm_OD2.1mm, symbol Connector:Conn_01x01_Pin
Connections:
- net MOTOR 1 +: now also J1.1 (Pin_1)
- net MOTOR 1 -: now also J2.1 (Pin_1)
- net MOTOR 2 +: now also J3.1 (Pin_1)
- net MOTOR 2 -: now also J4.1 (Pin_1)

Commit message: PCB smd - schematic update
Parts:
- removed J1, J2, J3, J4: Conn_01x01_Pin, Connector_Wire:SolderWire-0.5sqmm_1x01_D0.9mm_OD2.1mm, symbol Connector:Conn_01x01_Pin
- added J1: Conn_01x04_Pin, Connector_PinHeader_2.54mm:PinHeader_1x04_P2.54mm_Vertical, symbol Connector:Conn_01x04_Pin
Connections:
- net MOTOR 1 +: now also J1.1 (Pin_1)
- net MOTOR 1 -: now also J1.2 (Pin_2)
- net MOTOR 2 +: now also J1.4 (Pin_4)
- net MOTOR 2 -: now also J1.3 (Pin_3)
Changed lines of the file:
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@@
     (effects (font (size 1.27 1.27) italic) (justify left bottom))
   )
-  (global_label "MOTOR 1 +" (shape input) (at 170.18 118.11 0) (fields_autoplaced)
-    (effects (font (size 1.27 1.27)) (justify left))
-    (property "Intersheetrefs" "${INTERSHEET_REFS}" (at 184.1529 118.11 0)
-      (effects (font (size 1.27 1.27)) (justify left) hide)
-    )
-  )
-  (global_label "MOTOR 2 +" (shape input) (at 170.18 125.73 0) (fields_autoplaced)
-    (effects (font (size 1.27 1.27)) (justify left))
-    (property "Intersheetrefs" "${INTERSHEET_REFS}" (at 184.1529 125.73 0)
-      (effects (font (size 1.27 1.27)) (justify left) hide)
-    )
-  )
-  (global_label "MOTOR 2 -" (shape input) (at 170.18 129.54 0) (fields_autoplaced)
-    (effects (font (size 1.27 1.27)) (justify left))
-    (property "Intersheetrefs" "${INTERSHEET_REFS}" (at 184.1529 129.54 0)
-      (effects (font (size 1.27 1.27)) (justify left) hide)
-    )
-  )
-  (global_label "MOTOR 1 -" (shape input) (at 170.18 121.92 0) (fields_autoplaced)
-    (effects (font (size 1.27 1.27)) (justify left))
-    (property "Intersheetrefs" "${INTERSHEET_REFS}" (at 184.1529 121.92 0)
+  (global_label "MOTOR 1 +" (shape input) (at 176.53 118.11 0) (fields_autoplaced)
+    (effects (font (size 1 1)) (justify left))
+    (property "Intersheetrefs" "${INTERSHEET_REFS}" (at 187.5322 118.11 0)
+      (effects (font (size 1.27 1.27)) (justify left) hide)
+    )
+  )
+  (global_label "MOTOR 2 +" (shape input) (at 176.53 125.73 0) (fields_autoplaced)
+    (effects (font (size 1 1)) (justify left))
+    (property "Intersheetrefs" "${INTERSHEET_REFS}" (at 187.5322 125.73 0)
+      (effects (font (size 1.27 1.27)) (justify left) hide)
+    )
+  )
+  (global_label "MOTOR 2 -" (shape input) (at 176.53 123.19 0) (fields_autoplaced)
+    (effects (font (size 1 1)) (justify left))
+    (property "Intersheetrefs" "${INTERSHEET_REFS}" (at 187.5322 123.19 0)
+      (effects (font (size 1.27 1.27)) (justify left) hide)
+    )
+  )
+  (global_label "MOTOR 1 -" (shape input) (at 176.53 120.65 0) (fields_autoplaced)
+    (effects (font (size 1 1)) (justify left))
+    (property "Intersheetrefs" "${INTERSHEET_REFS}" (at 187.5322 120.65 0)
       (effects (font (size 1.27 1.27)) (justify left) hide)
     )
@@
     )
   )
-  (symbol (lib_id "Connector:Conn_01x01_Pin") (at 165.1 121.92 0) (unit 1)
-    (in_bom yes) (on_board yes) (dnp no)
-    (property "Reference" "J2" (at 162.56 121.92 0)
-      (effects (font (size 1.27 1.27)))
-    )
-    (property "Value" "Conn_01x01_Pin" (at 165.735 120.65 0)
-      (effects (font (size 1.27 1.27)) hide)
-    )
-    (property "Footprint" "Connector_Wire:SolderWire-0.5sqmm_1x01_D0.9mm_OD2.1mm" (at 165.1 121.92 0)
-      (effects (font (size 1.27 1.27)) hide)
-    )
-    (property "Datasheet" "~" (at 165.1 121.92 0)
-      (effects (font (size 1.27 1.27)) hide)
-    )
-    (pin "1")
-    (instances
-      (project "sumec"
-        (path "/fc70a1a8-ed7c-4a0f-9b1a-f23293528385/05a35bad-c108-46ad-8f95-76319a60a14f"
-          (reference "J2") (unit 1)
-        )
-      )
-    )
-  )
   (symbol (lib_id "Mechanical:MountingHole") (at 72.39 68.58 0) (unit 1)
     (in_bom yes) (on_board yes) (dnp no) (fields_autoplaced)
@@
     )
   )
+  (symbol (lib_id "Connector:Conn_01x04_Pin") (at 171.45 120.65 0) (unit 1)
+    (in_bom yes) (on_board yes) (dnp no)
+    (property "Reference" "J1" (at 168.91 121.92 0)
+      (effects (font (size 1.27 1.27)))
+    )
+    (property "Value" "Conn_01x04_Pin" (at 172.085 116.84 0)
+      (effects (font (size 1.27 1.27)) hide)
+    )
+    (property "Footprint" "Connector_PinHeader_2.54mm:PinHeader_1x04_P2.54mm_Vertical" (at 171.45 120.65 0)
+      (effects (font (size 1.27 1.27)) hide)
+    )
+    (property "Datasheet" "~" (at 171.45 120.65 0)
+      (effects (font (size 1.27 1.27)) hide)
+    )
+    (pin "1")
+    (pin "2")
+    (pin "3")
+    (pin "4")
+    (instances
+      (project "sumec"
+        (path "/fc70a1a8-ed7c-4a0f-9b1a-f23293528385/05a35bad-c108-46ad-8f95-76319a60a14f"
+          (reference "J1") (unit 1)
+        )
+      )
+    )
+  )
   (symbol (lib_id "power:+3V3") (at 86.36 130.81 90) (unit 1)
     (in_bom yes) (on_board yes) (dnp no) (fields_autoplaced)
@@
         (path "/fc70a1a8-ed7c-4a0f-9b1a-f23293528385/05a35bad-c108-46ad-8f95-76319a60a14f"
           (reference "#PWR02") (unit 1)
-        )
-      )
-    )
-  )
-  (symbol (lib_id "Connector:Conn_01x01_Pin") (at 165.1 125.73 0) (unit 1)
-    (in_bom yes) (on_board yes) (dnp no)
-    (property "Reference" "J3" (at 162.56 125.73 0)
-      (effects (font (size 1.27 1.27)))
-    )
-    (property "Value" "Conn_01x01_Pin" (at 165.735 124.46 0)
-      (effects (font (size 1.27 1.27)) hide)
-    )
-    (property "Footprint" "Connector_Wire:SolderWire-0.5sqmm_1x01_D0.9mm_OD2.1mm" (at 165.1 125.73 0)
-      (effects (font (size 1.27 1.27)) hide)
-    )
-    (property "Datasheet" "~" (at 165.1 125.73 0)
-      (effects (font (size 1.27 1.27)) hide)
-    )
-    (pin "1")
-    (instances
-      (project "sumec"
-        (path "/fc70a1a8-ed7c-4a0f-9b1a-f23293528385/05a35bad-c108-46ad-8f95-76319a60a14f"
-          (reference "J3") (unit 1)
         )
       )
@@
         (path "/fc70a1a8-ed7c-4a0f-9b1a-f23293528385/05a35bad-c108-46ad-8f95-76319a60a14f"
           (reference "H1") (unit 1)
-        )
-      )
-    )
-  )
-  (symbol (lib_id "Connector:Conn_01x01_Pin") (at 165.1 118.11 0) (unit 1)
-    (in_bom yes) (on_board yes) (dnp no)
-    (property "Reference" "J1" (at 162.56 118.11 0)
-      (effects (font (size 1.27 1.27)))
-    )
-    (property "Value" "Conn_01x01_Pin" (at 165.735 116.84 0)
-      (effects (font (size 1.27 1.27)) hide)
-    )
-    (property "Footprint" "Connector_Wire:SolderWire-0.5sqmm_1x01_D0.9mm_OD2.1mm" (at 165.1 118.11 0)
-      (effects (font (size 1.27 1.27)) hide)
-    )
-    (property "Datasheet" "~" (at 165.1 118.11 0)
-      (effects (font (size 1.27 1.27)) hide)
-    )
-    (pin "1")
-    (instances
-      (project "sumec"
-        (path "/fc70a1a8-ed7c-4a0f-9b1a-f23293528385/05a35bad-c108-46ad-8f95-76319a60a14f"
-          (reference "J1") (unit 1)
         )
       )
@@
         )
       )
-    )
-  )
-  (symbol (lib_id "Connector:Conn_01x01_Pin") (at 165.1 129.54 0) (unit 1)
-    (in_bom yes) (on_board yes) (dnp no)
-    (property "Reference" "J4" (at 162.56 129.54 0)
-      (effects (font (size 1.27 1.27)))
-    )
-    (property "Value" "Conn_01x01_Pin" (at 165.735 128.27 0)
-      (effects (font (size 1.27 1.27)) hide)
-    )
-    (property "Footprint" "Connector_Wire:SolderWire-0.5sqmm_1x01_D0.9mm_OD2.1mm" (at 165.1 129.54 0)
-      (effects (font (size 1.27 1.27)) hide)
-    )
-    (property "Datasheet" "~" (at 165.1 129.54 0)
-      (effects (font (size 1.27 1.27)) hide)
-    )
-    (pin "1")
-    (instances
-      (project "sumec"
-        (path "/fc70a1a8-ed7c-4a0f-9b1a-f23293528385/05a35bad-c108-46ad-8f95-76319a60a14f"
-          (reference "J4") (unit 1)
-        )
-      )

Commit message: PCB SMD - WIP ESP32 S3 WROOM 2
Parts:
- added H?: MountingHole M3, MountingHole:MountingHole_3.2mm_M3, symbol Mechanical:MountingHole
Connections:
- net +12V renamed +8V
- net 12V IN renamed 8V IN
Other:
- note added: "SPDT Switch 3 pin switch that works as a power-up lever Connected to the battery One pin is unused aprox. 1060mA 8,4V"
- note removed: "SPDT Switch 3 pin switch that works as a power-up lever Connected to the battery One pin is unused aprox. 1060mA 12,6 V Must take at least 13 volts and 1,5 amps."
- moved on the sheet: H?
Changed lines of the file:
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@@
     (effects (font (size 2 2)) (justify left bottom))
   )
-  (text "SPDT Switch\n\n3 pin switch that works as a power-up lever \nConnected to the battery \nOne pin is unused\n\naprox. 1060mA\n12,6 V\n\nMust take at least 13 volts and 1,5 amps."
-    (at 149.86 67.31 0)
+  (text "SPDT Switch\n\n3 pin switch that works as a power-up lever \nConnected to the battery \nOne pin is unused\n\naprox. 1060mA\n8,4V\n\n"
+    (at 151.13 66.04 0)
     (effects (font (size 1.3 1.3) italic) (justify left bottom))
   )
@@
   )
   (text "Mounting holes M3 \n\nMounting holes that are screwed \nto the heat-inserts on the chassis\n"
-    (at 67.31 55.88 0)
+    (at 67.31 68.58 0)
     (effects (font (size 1.5 1.5) italic) (justify left bottom))
   )
@@
     )
   )
-  (global_label "12V IN" (shape input) (at 180.34 78.74 0) (fields_autoplaced)
+  (global_label "8V IN" (shape input) (at 180.34 78.74 0) (fields_autoplaced)
     (effects (font (size 1.27 1.27)) (justify left))
-    (property "Intersheetrefs" "${INTERSHEET_REFS}" (at 189.4507 78.74 0)
-      (effects (font (size 1.27 1.27)) (justify left) hide)
-    )
-  )
-  (symbol (lib_id "Mechanical:MountingHole") (at 72.39 68.58 0) (unit 1)
-    (in_bom yes) (on_board yes) (dnp no) (fields_autoplaced)
-    (property "Reference" "H?" (at 74.93 67.945 0)
-      (effects (font (size 1.27 1.27)) (justify left))
-    )
-    (property "Value" "MountingHole M3" (at 74.93 70.485 0)
-      (effects (font (size 1.27 1.27)) (justify left))
-    )
-    (property "Footprint" "MountingHole:MountingHole_3.2mm_M3" (at 72.39 68.58 0)
-      (effects (font (size 1.27 1.27)) hide)
-    )
-    (property "Datasheet" "~" (at 72.39 68.58 0)
+    (property "Intersheetrefs" "${INTERSHEET_REFS}" (at 188.4468 78.74 0)
+      (effects (font (size 1.27 1.27)) (justify left) hide)
+    )
+  )
+  (symbol (lib_id "Mechanical:MountingHole") (at 118.11 62.23 0) (unit 1)
+    (in_bom yes) (on_board yes) (dnp no) (fields_autoplaced)
+    (property "Reference" "H?" (at 120.65 61.595 0)
+      (effects (font (size 1.27 1.27)) (justify left))
+    )
+    (property "Value" "MountingHole M3" (at 120.65 64.135 0)
+      (effects (font (size 1.27 1.27)) (justify left))
+    )
+    (property "Footprint" "MountingHole:MountingHole_3.2mm_M3" (at 118.11 62.23 0)
+      (effects (font (size 1.27 1.27)) hide)
+    )
+    (property "Datasheet" "~" (at 118.11 62.23 0)
       (effects (font (size 1.27 1.27)) hide)
     )
@@
     )
   )
-  (symbol (lib_id "Mechanical:MountingHole") (at 72.39 76.2 0) (unit 1)
-    (in_bom yes) (on_board yes) (dnp no) (fields_autoplaced)
-    (property "Reference" "H?" (at 74.93 75.565 0)
-      (effects (font (size 1.27 1.27)) (justify left))
-    )
-    (property "Value" "MountingHole M3" (at 74.93 78.105 0)
-      (effects (font (size 1.27 1.27)) (justify left))
-    )
-    (property "Footprint" "MountingHole:MountingHole_3.2mm_M3" (at 72.39 76.2 0)
-      (effects (font (size 1.27 1.27)) hide)
-    )
-    (property "Datasheet" "~" (at 72.39 76.2 0)
+  (symbol (lib_id "Mechanical:MountingHole") (at 118.11 69.85 0) (unit 1)
+    (in_bom yes) (on_board yes) (dnp no) (fields_autoplaced)
+    (property "Reference" "H?" (at 120.65 69.215 0)
+      (effects (font (size 1.27 1.27)) (justify left))
+    )
+    (property "Value" "MountingHole M3" (at 120.65 71.755 0)
+      (effects (font (size 1.27 1.27)) (justify left))
+    )
+    (property "Footprint" "MountingHole:MountingHole_3.2mm_M3" (at 118.11 69.85 0)
+      (effects (font (size 1.27 1.27)) hide)
+    )
+    (property "Datasheet" "~" (at 118.11 69.85 0)
       (effects (font (size 1.27 1.27)) hide)
     )
@@
     )
   )
+  (symbol (lib_id "Mechanical:MountingHole") (at 118.11 77.47 0) (unit 1)
+    (in_bom yes) (on_board yes) (dnp no) (fields_autoplaced)
+    (property "Reference" "H?" (at 120.65 76.835 0)
+      (effects (font (size 1.27 1.27)) (justify left))
+    )
+    (property "Value" "MountingHole M3" (at 120.65 79.375 0)
+      (effects (font (size 1.27 1.27)) (justify left))
+    )
+    (property "Footprint" "MountingHole:MountingHole_3.2mm_M3" (at 118.11 77.47 0)
+      (effects (font (size 1.27 1.27)) hide)
+    )
+    (property "Datasheet" "~" (at 118.11 77.47 0)
+      (effects (font (size 1.27 1.27)) hide)
+    )
+    (instances
+      (project "sumec"
+        (path "/fc70a1a8-ed7c-4a0f-9b1a-f23293528385"
+          (reference "H?") (unit 1)
+        )
+        (path "/fc70a1a8-ed7c-4a0f-9b1a-f23293528385/05a35bad-c108-46ad-8f95-76319a60a14f"
+          (reference "H4") (unit 1)
+        )
+      )
+    )
+  )
   (symbol (lib_id "power:+3V3") (at 86.36 130.81 90) (unit 1)
     (in_bom yes) (on_board yes) (dnp no) (fields_autoplaced)
@@
     )
   )
-  (symbol (lib_id "Mechanical:MountingHole") (at 72.39 60.96 0) (unit 1)
-    (in_bom yes) (on_board yes) (dnp no) (fields_autoplaced)
-    (property "Reference" "H?" (at 74.93 60.325 0)
-      (effects (font (size 1.27 1.27)) (justify left))
-    )
-    (property "Value" "MountingHole M3" (at 74.93 62.865 0)
-      (effects (font (size 1.27 1.27)) (justify left))
-    )
-    (property "Footprint" "MountingHole:MountingHole_3.2mm_M3" (at 72.39 60.96 0)
-      (effects (font (size 1.27 1.27)) hide)
-    )
-    (property "Datasheet" "~" (at 72.39 60.96 0)
+  (symbol (lib_id "power:+8V") (at 165.1 76.2 90) (unit 1)
+    (in_bom yes) (on_board yes) (dnp no) (fields_autoplaced)
+    (property "Reference" "#PWR038" (at 168.91 76.2 0)
+      (effects (font (size 1.27 1.27)) hide)
+    )
+    (property "Value" "+8V" (at 161.29 76.835 90)
+      (effects (font (size 1.27 1.27)) (justify left))
+    )
+    (property "Footprint" "" (at 165.1 76.2 0)
+      (effects (font (size 1.27 1.27)) hide)
+    )
+    (property "Datasheet" "" (at 165.1 76.2 0)
+      (effects (font (size 1.27 1.27)) hide)
+    )
+    (pin "1")
+    (instances
+      (project "sumec"
+        (path "/fc70a1a8-ed7c-4a0f-9b1a-f23293528385/05a35bad-c108-46ad-8f95-76319a60a14f"
+          (reference "#PWR038") (unit 1)
+        )
+      )
+    )
+  )
+  (symbol (lib_id "Mechanical:MountingHole") (at 118.11 54.61 0) (unit 1)
+    (in_bom yes) (on_board yes) (dnp no) (fields_autoplaced)
+    (property "Reference" "H?" (at 120.65 53.975 0)
+      (effects (font (size 1.27 1.27)) (justify left))
+    )
+    (property "Value" "MountingHole M3" (at 120.65 56.515 0)
+      (effects (font (size 1.27 1.27)) (justify left))
+    )
+    (property "Footprint" "MountingHole:MountingHole_3.2mm_M3" (at 118.11 54.61 0)
+      (effects (font (size 1.27 1.27)) hide)
+    )
+    (property "Datasheet" "~" (at 118.11 54.61 0)
       (effects (font (size 1.27 1.27)) hide)
     )
@@
         )
       )
-    )
-  )
-  (symbol (lib_id "power:+12V") (at 165.1 76.2 90) (mirror x) (unit 1)
-    (in_bom yes) (on_board yes) (dnp no)
-    (property "Reference" "#PWR?" (at 168.91 76.2 0)
-      (effects (font (size 1.27 1.27)) hide)
-    )
-    (property "Value" "+12V" (at 158.75 76.2 90)
-      (effects (font (size 1.27 1.27)))
-    )
-    (property "Footprint" "Battery:BatteryHolder_Bulgin_BX0036_1xC" (at 165.1 76.2 0)
-      (effects (font (size 1.27 1.27)) hide)
-    )
-    (property "Datasheet" "" (at 165.1 76.2 0)
-      (effects (font (size 1.27 1.27)) hide)
-    )
-    (pin "1")
-    (instances
-      (project "sumec"
-        (path "/fc70a1a8-ed7c-4a0f-9b1a-f23293528385"
-          (reference "#PWR?") (unit 1)
-        )
-        (path "/fc70a1a8-ed7c-4a0f-9b1a-f23293528385/05a35bad-c108-46ad-8f95-76319a60a14f"
-          (reference "#PWR038") (unit 1)
-        )
-      )

Commit message: i desire sleep
Connections:
- net MOTOR 2 +: now also J1.3 (Pin_3); no longer J1.4 (Pin_4)
- net MOTOR 2 -: now also J1.4 (Pin_4); no longer J1.3 (Pin_3)
Changed lines of the file:
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@@
-    )
-  )
-  (global_label "MOTOR 2 +" (shape input) (at 176.53 125.73 0) (fields_autoplaced)
-    (effects (font (size 1 1)) (justify left))
-    (property "Intersheetrefs" "${INTERSHEET_REFS}" (at 187.5322 125.73 0)
-      (effects (font (size 1.27 1.27)) (justify left) hide)
-    )
-  )
-  (global_label "MOTOR 2 -" (shape input) (at 176.53 123.19 0) (fields_autoplaced)
-    (effects (font (size 1 1)) (justify left))
-    (property "Intersheetrefs" "${INTERSHEET_REFS}" (at 187.5322 123.19 0)
-      (effects (font (size 1.27 1.27)) (justify left) hide)
     )
   )
@@
     )
   )
+  (global_label "MOTOR 2 +" (shape input) (at 176.53 123.19 0) (fields_autoplaced)
+    (effects (font (size 1 1)) (justify left))
+    (property "Intersheetrefs" "${INTERSHEET_REFS}" (at 187.5322 123.19 0)
+      (effects (font (size 1.27 1.27)) (justify left) hide)
+    )
+  )
   (global_label "8V IN" (shape input) (at 180.34 78.74 0) (fields_autoplaced)
     (effects (font (size 1.27 1.27)) (justify left))
@@
     )
   )
+  (global_label "MOTOR 2 -" (shape input) (at 176.53 125.73 0) (fields_autoplaced)
+    (effects (font (size 1 1)) (justify left))
+    (property "Intersheetrefs" "${INTERSHEET_REFS}" (at 187.5322 125.73 0)
+      (effects (font (size 1.27 1.27)) (justify left) hide)
+    )
+  )
   (symbol (lib_id "Mechanical:MountingHole") (at 118.11 62.23 0) (unit 1)
-    (in_bom yes) (on_board yes) (dnp no) (fields_autoplaced)
+    (in_bom yes) (on_board yes) (dnp no)
     (property "Reference" "H?" (at 120.65 61.595 0)
-      (effects (font (size 1.27 1.27)) (justify left))
-    )
-    (property "Value" "MountingHole M3" (at 120.65 64.135 0)
+      (effects (font (size 1.27 1.27)) (justify left) hide)
+    )
+    (property "Value" "MountingHole M3" (at 120.65 62.23 0)
       (effects (font (size 1.27 1.27)) (justify left))
     )
@@
   )
   (symbol (lib_id "Mechanical:MountingHole") (at 118.11 69.85 0) (unit 1)
-    (in_bom yes) (on_board yes) (dnp no) (fields_autoplaced)
+    (in_bom yes) (on_board yes) (dnp no)
     (property "Reference" "H?" (at 120.65 69.215 0)
-      (effects (font (size 1.27 1.27)) (justify left))
-    )
-    (property "Value" "MountingHole M3" (at 120.65 71.755 0)
+      (effects (font (size 1.27 1.27)) (justify left) hide)
+    )
+    (property "Value" "MountingHole M3" (at 120.65 69.85 0)
       (effects (font (size 1.27 1.27)) (justify left))
     )
@@
   )
   (symbol (lib_id "Mechanical:MountingHole") (at 118.11 77.47 0) (unit 1)
-    (in_bom yes) (on_board yes) (dnp no) (fields_autoplaced)
+    (in_bom yes) (on_board yes) (dnp no)
     (property "Reference" "H?" (at 120.65 76.835 0)
-      (effects (font (size 1.27 1.27)) (justify left))
-    )
-    (property "Value" "MountingHole M3" (at 120.65 79.375 0)
+      (effects (font (size 1.27 1.27)) (justify left) hide)
+    )
+    (property "Value" "MountingHole M3" (at 120.65 77.47 0)
       (effects (font (size 1.27 1.27)) (justify left))
     )
@@
   )
   (symbol (lib_id "Mechanical:MountingHole") (at 118.11 54.61 0) (unit 1)
-    (in_bom yes) (on_board yes) (dnp no) (fields_autoplaced)
+    (in_bom yes) (on_board yes) (dnp no)
     (property "Reference" "H?" (at 120.65 53.975 0)
-      (effects (font (size 1.27 1.27)) (justify left))
-    )
-    (property "Value" "MountingHole M3" (at 120.65 56.515 0)
-      (effects (font (size 1.27 1.27)) (justify left))
-    )
+      (effects (font (size 1.27 1.27)) (justify left) hide)
+    )
+    (property "Value" "MountingHole M3" (at 120.65 54.61 0)
+      (effects (font (size 1.27 1.27)) (justify left))
+    )
