File: - PCB -/SUMEC SMD/MCU.kicad_sch (KiCad schematic)
At the start: 24 parts, among them J2 USB3090-XX-X_REVE, Q3 PMOS, SW2 SW_Push, SW4 SW_Push, U10 TB6612FNG, U9 ESP32-S3-WROOM-1

Commit message: pcb board development (cool)
Parts:
- Q3: footprint Package_TO_SOT_THT:TO-220-3_Vertical -> Package_TO_SOT_SMD:SOT-223
- SW2, SW4: footprint Button_Switch_THT:SW_PUSH_6mm -> Button_Switch_SMD:SW_SPST_B3U-1000P
Connections:
- net PWMA: now also U9.24 (GPIO47/SPICLK_P/SUBSPICLK_P_DIFF); no longer U9.35 (MTMS/GPIO42)
- net PWMB: now also U9.23 (GPIO21); no longer U9.34 (MTDI/GPIO41/CLK_OUT1)
Changed lines of the file:
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@@
   (no_connect (at 297.18 189.23))
   (no_connect (at 285.75 219.71))
-  (no_connect (at 299.72 222.25))
   (no_connect (at 293.37 153.67))
   (no_connect (at 294.64 176.53))
   (no_connect (at 171.45 222.25))
+  (no_connect (at 179.07 173.99))
   (no_connect (at 185.42 163.83))
   (no_connect (at 171.45 224.79))
+  (no_connect (at 179.07 176.53))
   (no_connect (at 175.26 168.91))
   (no_connect (at 293.37 156.21))
@@
   (no_connect (at 185.42 161.29))
   (no_connect (at 447.04 140.97))
-  (no_connect (at 302.26 212.09))
   (no_connect (at 447.04 133.35))
   (no_connect (at 285.75 217.17))
@@
     (effects (font (size 1 1)) (justify right bottom))
   )
+  (label "PWMA" (at 299.72 222.25 180) (fields_autoplaced)
+    (effects (font (size 1 1)) (justify right bottom))
+  )
   (label "BOOT" (at 294.64 168.91 180) (fields_autoplaced)
     (effects (font (size 1 1)) (justify right bottom))
@@
     (effects (font (size 1 1)) (justify right bottom))
   )
-  (label "PWMA" (at 179.07 176.53 0) (fields_autoplaced)
-    (effects (font (size 1 1)) (justify left bottom))
-  )
   (label "VM" (at 177.8 353.06 90) (fields_autoplaced)
     (effects (font (size 1 1)) (justify left bottom))
   )
+  (label "PWMB" (at 302.26 212.09 180) (fields_autoplaced)
+    (effects (font (size 1 1)) (justify right bottom))
+  )
   (label "BI1" (at 299.72 201.93 180) (fields_autoplaced)
     (effects (font (size 1 1)) (justify right bottom))
@@
   (label "AI1" (at 207.01 317.5 180) (fields_autoplaced)
     (effects (font (size 1 1)) (justify right bottom))
-  )
-  (label "PWMB" (at 179.07 173.99 0) (fields_autoplaced)
-    (effects (font (size 1 1)) (justify left bottom))
   )
   (label "BOOT" (at 518.16 210.82 180) (fields_autoplaced)
@@
       (effects (font (size 1.27 1.27)))
     )
-    (property "Footprint" "Button_Switch_THT:SW_PUSH_6mm" (at 506.73 205.74 0)
+    (property "Footprint" "Button_Switch_SMD:SW_SPST_B3U-1000P" (at 506.73 205.74 0)
       (effects (font (size 1.27 1.27)) hide)
     )
@@
     )
   )
+  (symbol (lib_id "power:+3V3") (at 187.96 354.33 180) (unit 1)
+    (in_bom yes) (on_board yes) (dnp no)
+    (property "Reference" "#PWR?" (at 187.96 350.52 0)
+      (effects (font (size 1.27 1.27)) hide)
+    )
+    (property "Value" "+3V3" (at 187.96 358.14 90)
+      (effects (font (size 1.27 1.27)) (justify left))
+    )
+    (property "Footprint" "" (at 187.96 354.33 0)
+      (effects (font (size 1.27 1.27)) hide)
+    )
+    (property "Datasheet" "" (at 187.96 354.33 0)
+      (effects (font (size 1.27 1.27)) hide)
+    )
+    (pin "1")
+    (instances
+      (project "sumec"
+        (path "/fc70a1a8-ed7c-4a0f-9b1a-f23293528385"
+          (reference "#PWR?") (unit 1)
+        )
+        (path "/fc70a1a8-ed7c-4a0f-9b1a-f23293528385/2febd48c-c6ec-477b-ac64-6fa98a41fff0"
+          (reference "#PWR028") (unit 1)
+        )
+        (path "/fc70a1a8-ed7c-4a0f-9b1a-f23293528385/11aa20d4-c4ff-49be-9179-c2911da50f67"
+          (reference "#PWR011") (unit 1)
+        )
+      )
+    )
+  )
   (symbol (lib_id "Device:C") (at 506.73 217.17 270) (mirror x) (unit 1)
     (in_bom yes) (on_board yes) (dnp no)
@@
       (effects (font (size 1.27 1.27)))
     )
-    (property "Footprint" "Button_Switch_THT:SW_PUSH_6mm" (at 483.87 205.74 0)
+    (property "Footprint" "Button_Switch_SMD:SW_SPST_B3U-1000P" (at 483.87 205.74 0)
       (effects (font (size 1.27 1.27)) hide)
     )
@@
       (effects (font (size 1.27 1.27)))
     )
-    (property "Footprint" "Package_TO_SOT_THT:TO-220-3_Vertical" (at 228.6 298.45 0)
+    (property "Footprint" "Package_TO_SOT_SMD:SOT-223" (at 228.6 298.45 0)
       (effects (font (size 1.27 1.27)) hide)
     )
@@
         )
       )
-    )
-  )
-  (symbol (lib_name "+3V3_1") (lib_id "power:+3V3") (at 187.96 354.33 180) (unit 1)
-    (in_bom yes) (on_board yes) (dnp no)
-    (property "Reference" "#PWR?" (at 187.96 350.52 0)
-      (effects (font (size 1.27 1.27)) hide)
-    )
-    (property "Value" "+3V3" (at 184.15 355.6 0)
-      (effects (font (size 1.27 1.27)))
-    )
-    (property "Footprint" "" (at 187.96 354.33 0)
-      (effects (font (size 1.27 1.27)) hide)
-    )
-    (property "Datasheet" "" (at 187.96 354.33 0)
-      (effects (font (size 1.27 1.27)) hide)
-    )
-    (pin "1")
-    (instances
-      (project "sumec"
-        (path "/fc70a1a8-ed7c-4a0f-9b1a-f23293528385"
-          (reference "#PWR?") (unit 1)
-        )
-        (path "/fc70a1a8-ed7c-4a0f-9b1a-f23293528385/2febd48c-c6ec-477b-ac64-6fa98a41fff0"
-          (reference "#PWR032") (unit 1)
-        )
-        (path "/fc70a1a8-ed7c-4a0f-9b1a-f23293528385/11aa20d4-c4ff-49be-9179-c2911da50f67"
-          (reference "#PWR011") (unit 1)
-        )
-      )

Commit message: PCB schematic update
Parts:
- removed C?: 0,5uF.hbc, Capacitor_SMD:C_1206_3216Metric, symbol Device:C
- removed D2, D3, D4, D5: ESD5Zxx, Diode_SMD:D_SOD-523, symbol Diode:ESD5Zxx
- removed D7.hbc1: D_Zener, Diode_SMD:D_1206_3216Metric, symbol Device:D_Zener
- removed Q3: PMOS, Package_TO_SOT_SMD:SOT-223, symbol Simulation_SPICE:PMOS
- removed R25: 100k.hbc, Resistor_SMD:R_1206_3216Metric, symbol Device:R
- added C5: 100nF, symbol Device:C
- added R2, R3: 15R, symbol Device:R
- added R6: 0R, symbol Device:R
- added U2: USBLC6-2SC6, USBLC6-2SC6:SOT95P280X145-6N, symbol sumec_library:USBLC6-2SC6
- C?: value 0,1uF.mcu -> 100nF.mcu
- C?: value 0,1uF.hbc -> 100nF.hbc
- C?: value 0,1uF.boot -> 100nF.boot
- C?: value 0,1uF.en -> 100nF.en
Connections:
- net VM is gone; now on net +8V: C?.1, C?.1, U10.13 (VM2), U10.14 (VM3), U10.24 (VM1)
- net GND: now also C5.2, R6.2, U2.2
- net at J2.6 (SHIELD), J2.7 (SHIELD), J2.8 (SHIELD)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: now also R6.1
- net +5V renamed VBUS 5V
- net VBUS 5V: now also C5.1, U2.5
- net D +: no longer names the net of J2.3 (D+)
- net D +: now also R2.1; no longer U9.14 (GPIO20/U1CTS/ADC2_CH9/CLK_OUT1/USB_D+)
- net D -: no longer names the net of J2.2 (D-)
- net D -: now also R3.1; no longer U9.13 (GPIO19/U1RTS/ADC2_CH8/CLK_OUT2/USB_D-)
- net QRE1113 A: no longer names the net of U9.4 (GPIO4/TOUCH4/ADC1_CH3)
- new net: R2.2, U2.1
- new net: R3.2, U2.3
- new net D+: U2.6, U9.14 (GPIO20/U1CTS/ADC2_CH9/CLK_OUT1/USB_D+)
- new net D-: U2.4, U9.13 (GPIO19/U1RTS/ADC2_CH8/CLK_OUT2/USB_D-)
- no-connect marks 18 -> 20
Other:
- note added: "ESD PROTECTION"
- note removed: "ESD protection"
- note removed: "není toho hodně? mohli bysme to ulehčit."
- moved on the sheet: C?, J2

Commit message: pcb scheamtic and board update
Parts:
- removed J2: USB3090-XX-X_REVE, sumec-smd_library:GCT_USB3090-XX-X_REVE, symbol sumec_library:USB3090-XX-X_REVE
- added J2: TYPE-C-31-M-12, TYPE-C-31-M-12:HRO_TYPE-C-31-M-12, symbol sumec_library:TYPE-C-31-M-12
- C5: footprint (none) -> Capacitor_SMD:C_1206_3216Metric
- R2, R3, R6: footprint (none) -> Resistor_SMD:R_1206_3216Metric
- U2: footprint USBLC6-2SC6:SOT95P280X145-6N -> Package_TO_SOT_SMD:TSOT-23-6_HandSoldering
Connections:
- net GND: now also J2.A1_B12 (GND), J2.B1_A12 (GND)
- net at D1.2 (A): now also J2.A4_B9 (VBUS), J2.B4_A9 (VBUS)
- net at R3.1: now also J2.A7 (DN1)
- net at R2.1: now also J2.A6 (DP1)
- net at R6.1: now also J2.S1 (SHIELD), J2.S2 (SHIELD), J2.S3 (SHIELD), J2.S4 (SHIELD)
- no-connect marks 20 -> 25
Other:
- moved on the sheet: C5, D1, R2, R3, U2
