File: - PCB -/SUMEC SMD updated/POWER SUPPLY.kicad_sch (KiCad schematic)
At the start: 7 parts, among them U7 LM1084IS-5.0/NOPB, U8 LM1084IS-3.3/NOPB

Commit message: cleanup sumec enchanced
Parts:
- removed C? (x4): 10uF.stabl, Capacitor_SMD:C_1206_3216Metric_Pad1.33x1.80mm_HandSolder, symbol Device:C
- added C10, C11, C12, C13: 10uF.stabl, symbol Device:C_Polarized
- U7: footprint Package_TO_SOT_SMD:TO-252-3_TabPin2 -> Package_TO_SOT_SMD:TO-263-3_TabPin4
Connections:
- net +3V3: now also C13.1
- net +5V: now also C11.1, C12.1
- net +8V: now also C10.1
- net GND: now also C10.2, C11.2, C12.2, C13.2
Other:
- note removed: "Voltage stabilaser LM1084 Input voltage 8,4V Voltage regulator - 3,3V Output current - 5A"
