File: - PCB -/SUMEC SMD Encahnced/sumec.kicad_sch (KiCad schematic)
At the start: 2 parts

Commit message: Revert "Merge branch 'sumec-main' of https://github.com/menmenson/RoboCop into sumec-main"
This reverts commit dbf205ac3b02d72b1b38e86a27b286e1b118f9d4, reversing
changes made to f2387d167bca73d6a0741a06b82f65a42dfb555a.
Parts:
- R1, R2: value ~ -> R
Changed lines of the file:
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@@
   )
   (text "ESP32-S3 Datasheet" (at 115.57 127 0)
-    (effects (font (size 5 5) (thickness 1) bold (color 0 0 0 1)) (justify left bottom) (href "https://www.espressif.com/sites/default/files/documentation/esp32-s3_datasheet_en.pdf"))
+    (effects (font (size 5 5) (thickness 1) bold) (justify left bottom) (href "https://www.espressif.com/sites/default/files/documentation/esp32-s3_datasheet_en.pdf"))
   )
   (symbol (lib_id "Device:R") (at 153.67 40.64 90) (unit 1)
@@
       (effects (font (size 1.27 1.27)) hide)
     )
-    (property "Value" "~" (at 153.67 38.1 90)
+    (property "Value" "R" (at 153.67 38.1 90)
       (effects (font (size 1.27 1.27)) hide)
     )
@@
       (effects (font (size 1.27 1.27)) hide)
     )
-    (property "Value" "~" (at 153.67 34.29 90)
+    (property "Value" "R" (at 153.67 34.29 90)
       (effects (font (size 1.27 1.27)) hide)
     )

Commit message: QRE Array - WIP
Parts:
- R1, R2: value R -> ~
Changed lines of the file:
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@@
   )
   (text "ESP32-S3 Datasheet" (at 115.57 127 0)
-    (effects (font (size 5 5) (thickness 1) bold) (justify left bottom) (href "https://www.espressif.com/sites/default/files/documentation/esp32-s3_datasheet_en.pdf"))
+    (effects (font (size 5 5) (thickness 1) bold (color 0 0 0 1)) (justify left bottom) (href "https://www.espressif.com/sites/default/files/documentation/esp32-s3_datasheet_en.pdf"))
   )
   (symbol (lib_id "Device:R") (at 153.67 40.64 90) (unit 1)
@@
       (effects (font (size 1.27 1.27)) hide)
     )
-    (property "Value" "R" (at 153.67 38.1 90)
+    (property "Value" "~" (at 153.67 38.1 90)
       (effects (font (size 1.27 1.27)) hide)
     )
@@
       (effects (font (size 1.27 1.27)) hide)
     )
-    (property "Value" "R" (at 153.67 34.29 90)
+    (property "Value" "~" (at 153.67 34.29 90)
       (effects (font (size 1.27 1.27)) hide)
     )
