File: - PCB -/SUMEC SMD Encahnced/sumec.kicad_pcb (KiCad board)
At the start: 2 copper layers, 92 x 56.5 mm, 60 parts, among them IC1 XT30U-F, J1 Conn_01x04_Pin, J2 Conn_01x01_Pin, J3 Conn_01x03_Pin, J4 Conn_01x02, J5 TYPE-C-31-M-12, J6 Conn_01x06_Pin, J7 Conn_01x06_Pin, J8 TSOP382xx, J9 Conn_01x06_Pin, SW1 SW_Push, SW2 SW_Push, SW3 SW_Push, U1 TB6612FNG, U2 ESP32-S3-WROOM-1, U3 USBLC6-2SC6, U4 QRE1113, U5 QRE1113, U6 QRE1113, U7 LM1084IS-5.0/NOPB, U8 LM1084IS-3.3/NOPB

Commit message: Pcb updates
Parts:
- U7, U8: footprint Package_TO_SOT_SMD:TO-252-3_TabPin2 -> Package_TO_SOT_SMD:TO-263-3_TabPin4
- moved U7 42.9 mm to (228.9, 46.7), turned to 90 degrees
- moved U8 26.8 mm to (243.7, 28.1), turned to 90 degrees
Routing:
- net GND: vias 13 -> 14
- net +8V: vias 2 -> 3
- net +5V: vias 13 -> 11

Commit message: PCB Folder cleansing
Parts:
- removed C1: 10uF.hb, Capacitor_SMD:C_1206_3216Metric
- removed C10, C11, C12, C13: 10uF.stabl, Capacitor_SMD:C_1206_3216Metric_Pad1.33x1.80mm_HandSolder
- removed C2: 1uF.hb, Capacitor_SMD:C_1206_3216Metric
- removed C3: 10uF.mcu, Capacitor_SMD:C_1206_3216Metric
- removed C4: 100nF.mcu, Capacitor_SMD:C_1206_3216Metric
- removed C5: 10uF.hbc, Capacitor_SMD:C_1206_3216Metric
- removed C6: 100nF.hbc, Capacitor_SMD:C_1206_3216Metric
- removed C7: 100nF.en, Capacitor_SMD:C_1206_3216Metric
- removed C8: 100nF.boot, Capacitor_SMD:C_1206_3216Metric
- removed C9: 100nF, Capacitor_SMD:C_1206_3216Metric
- removed D1: LED, LED_SMD:LED_1206_3216Metric_Pad1.42x1.75mm_HandSolder
- removed D2: 1N5819, Diode_SMD:D_1206_3216Metric
- removed H1, H2, H3, H4: MountingHole M3, MountingHole:MountingHole_3.2mm_M3_ISO7380_Pad
- removed IC1: XT30U-F, sumec_library:AMASS_XT30U-M_1x02_P5.0mm_Vertical
- removed J1: Conn_01x04_Pin, Connector_PinHeader_2.54mm:PinHeader_1x04_P2.54mm_Vertical
- removed J2: Conn_01x01_Pin, Connector_Wire:SolderWire-0.1sqmm_1x01_D0.4mm_OD1mm
- removed J3: Conn_01x03_Pin, Connector_PinSocket_2.54mm:PinSocket_1x03_P2.54mm_Vertical
- removed J4: Conn_01x02, Connector_PinHeader_2.54mm:PinHeader_1x02_P2.54mm_Vertical
- removed J5: TYPE-C-31-M-12, sumec-smd_library:HRO_TYPE-C-31-M-12
- removed J6, J7, J9: Conn_01x06_Pin, Connector_JST:JST_SH_BM06B-SRSS-TB_1x06-1MP_P1.00mm_Vertical
- removed J8: TSOP382xx, Connector_PinSocket_2.54mm:PinSocket_1x03_P2.54mm_Vertical
- removed JP1: SolderJumper_3_Open, Jumper:SolderJumper-3_P2.0mm_Open_TrianglePad1.0x1.5mm
- removed R1: R, sumec-smd_library:logo even smaller
- removed R10, R11, R12, R13, R4, R8, R9: 0R, Resistor_SMD:R_1206_3216Metric
- removed R14, R16, R18: 100, Resistor_SMD:R_1206_3216Metric
- removed R15, R17, R19: 10k, Resistor_SMD:R_1206_3216Metric
- removed R2: R, sumec-smd_library:car cool smol
- removed R3: 220, Resistor_SMD:R_1206_3216Metric_Pad1.30x1.75mm_HandSolder
- removed R5, R6: 15R, Resistor_SMD:R_1206_3216Metric
- removed R7: 10k.mcu, Resistor_SMD:R_1206_3216Metric
- removed SW1, SW2, SW3: SW_Push, Button_Switch_SMD:SW_SPST_B3U-1000P
- removed U1: TB6612FNG, Package_SO:SSOP-24_5.3x8.2mm_P0.65mm
- removed U2: ESP32-S3-WROOM-1, PCM_Espressif:ESP32-S3-WROOM-1
- removed U3: USBLC6-2SC6, Package_TO_SOT_SMD:TSOT-23-6_HandSoldering
- removed U4, U5, U6: QRE1113, sumec_library:OnSemi_CASE100AQ - QRE1113
- removed U7: LM1084IS-5.0/NOPB, Package_TO_SOT_SMD:TO-263-3_TabPin4
- removed U8: LM1084IS-3.3/NOPB, Package_TO_SOT_SMD:TO-263-3_TabPin4
Routing:
- net +3V3: track 223.9 -> 0.00 mm, vias 19 -> 0
- net QRE1113 D: track 90.3 -> 0.00 mm, vias 2 -> 0
- net +8V: track 68.2 -> 0.00 mm, vias 3 -> 0
- net X-SHUT3: track 49.5 -> 0.00 mm, vias 2 -> 0
- net QRE1113 B: track 49.2 -> 0.00 mm, vias 2 -> 0
- net QRE1113 A: track 48.4 -> 0.00 mm, vias 2 -> 0
- net X-SHUT2: track 43.0 -> 0.00 mm, vias 2 -> 0
- net +5V: track 43.0 -> 0.00 mm, vias 11 -> 0
- net SCL: track 42.5 -> 0.00 mm, vias 2 -> 0
- net SDA: track 40.8 -> 0.00 mm, vias 2 -> 0
- net QRE1113 C: track 36.0 -> 0.00 mm, vias 1 -> 0
- net X-SHUT1: track 36.0 -> 0.00 mm, vias 2 -> 0
- net IR MODULE: track 23.0 -> 0.00 mm
- net MOTOR 1 +: track 19.8 -> 0.00 mm
- net SENSOR_SUPPLY: track 19.2 -> 0.00 mm
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- removed copper zone on B.Cu, net +3V3
- removed copper zone on B.Cu, net +5V
- removed copper zone on F.Cu, net +8V
- removed copper zone on B.Cu, net GND
- removed copper zone on F.Cu, net GND
- removed copper zone on F.Cu, net MOTOR 1 +
- removed copper zone on F.Cu, net MOTOR 1 -
- removed copper zone on F.Cu, net MOTOR 2 +
- removed copper zone on F.Cu, net MOTOR 2 -
Other:
- board outline removed
- board text removed: ">:3"
- board text removed: "BOOT"
- board text removed: "EN"
- board text removed: "TEST"
