File: - PCB -/Optic Lite-On Transistor/Optic Lite-On Transistor.kicad_sch (KiCad schematic)
At the start: 5 parts, among them J1 Conn_01x02_Pin, J3 Conn_01x04_Pin, U1 LTV-827

Commit message: Pcb updates
Other:
- moved on the sheet: J1, J3, R1, R2, U1A, U1B
