File: - PCB -/N-Channel Enhancement/N-Channel Enhancement.kicad_pcb (KiCad board)
At the start: 2 copper layers, 33.3 x 15.2 mm, 5 parts, among them J1 Conn_01x02_Pin, J3 Conn_01x04_Pin, U1 LTV-827

Commit message: matej push
Parts:
- removed U1: LTV-827, Package_DIP:DIP-8_W7.62mm
- added J2: Conn_01x03_Socket, Connector_PinSocket_2.54mm:PinSocket_1x03_P2.54mm_Vertical, F.Cu at (148.8, 38.2)
- added J4: Conn_01x03_Socket, Connector_PinSocket_2.54mm:PinSocket_1x03_P2.54mm_Vertical, F.Cu at (139.2, 49.0)
- added Q1: NMOS, Package_TO_SOT_SMD:SOT-23, B.Cu at (151.2, 43.8)
- added Q2: NMOS, Package_TO_SOT_SMD:SOT-23, B.Cu at (141.8, 43.8)
- J1: value Conn_01x02_Pin -> Conn_01x03_Socket; footprint Connector_JST:JST_XH_B2B-XH-A_1x02_P2.50mm_Vertical -> Connector_PinSocket_2.54mm:PinSocket_1x03_P2.54mm_Vertical
- J3: value Conn_01x04_Pin -> Conn_01x03_Socket; footprint Connector_JST:JST_XH_B4B-XH-A_1x04_P2.50mm_Vertical -> Connector_PinSocket_2.54mm:PinSocket_1x03_P2.54mm_Vertical
- R1, R2: value 210R -> 2.2k
- moved J1 81.4 mm to (148.8, 49.0), turned to 90 degrees
- moved J3 53.7 mm to (139.2, 38.2)
- moved R2 37.4 mm to (108.6, 55.8), turned to 0 degrees
- moved R1 34.9 mm to (108.6, 49.0), turned to 0 degrees
Connections:
- J1 pad 2: X-SHUT 1 -> TF-LUNA 2
- J3 pad 1: GND -> TF-LUNA 1
- J3 pad 2: TF-LUNA 2 -> X-SHUT 1
- R1 pad 1: X-SHUT 1 -> TF-LUNA 1
- R2 pad 1: X-SHUT 2 -> TF-LUNA 1
Routing:
- net GND: track 18.9 -> 0.00 mm
- net X-SHUT 1: track 14.3 -> 0.00 mm
- net SDA: track 10.3 -> 0.00 mm
- net Net-(Q2-D): track 10.1 -> 0.00 mm
- net X-SHUT 2: track 5.20 -> 0.00 mm
- net TF-LUNA 2: track 4.10 -> 0.00 mm
- net TF-LUNA 1: track 4.10 -> 0.00 mm
- net Net-(Q1-D): track 2.90 -> 0.00 mm
Other:
- board outline removed

Commit message: PCB Updates
Parts:
- added J5: Conn_01x01_Socket, Connector_PinSocket_2.54mm:PinSocket_1x01_P2.54mm_Vertical, F.Cu at (163.8, 30.2)
- J2, J4: value Conn_01x03_Socket -> Conn_01x01_Socket; footprint Connector_PinSocket_2.54mm:PinSocket_1x03_P2.54mm_Vertical -> Connector_PinSocket_2.54mm:PinSocket_1x01_P2.54mm_Vertical
- moved R2 50.5 mm to (158.2, 46.8), turned to 90 degrees
- moved R1 43.9 mm to (151.0, 37.8), turned to 180 degrees
- moved J4 23.2 mm to (152.5, 30.0), turned to 0 degrees
- moved J3 15.5 mm to (147.9, 25.4), turned to 0 degrees
- moved J2 13.4 mm to (152.5, 25.4), turned to 0 degrees
- moved J1 4.51 mm to (153.2, 49.2), turned to -90 degrees
- moved Q1 1.00 mm to (150.2, 43.8), turned to 90 degrees
- turned Q2 to 90 degrees
Connections:
- J1 pad 1: X-SHUT 2 -> TF-LUNA 1
- J1 pad 2: TF-LUNA 2 -> SDA
- J1 pad 3: SDA -> X-SHUT 2
- J2 pad 1: X-SHUT 2 -> SDA
- J3 pad 2: X-SHUT 1 -> SDA
- J3 pad 3: SDA -> X-SHUT 1
- J4 pad 1: TF-LUNA 1 -> SDA
