File: - PCB -/QRE MiniBoards/QRE MiniBoards.kicad_sch (KiCad schematic)
At the start: 9 parts, among them J2 Conn_01x04_Pin, Q1 PMOS, Q2 NMOS, U1 QRE1113, U2 QRE1113

Commit message: QRE MiniBoards - Finito
Parts:
- removed Q1: PMOS, symbol Simulation_SPICE:PMOS
- removed Q2: NMOS, symbol Simulation_SPICE:NMOS
- added H1, H2: MountingHole, MountingHole:MountingHole_3.2mm_M3_ISO7380_Pad, symbol Mechanical:MountingHole
Other:
- note added: "MECHANICAL"
- note added: "QRE1113 Sensors"
- moved on the sheet: J2, R1, R2, R3, R4, U1, U2

Commit message: QRE MiniBoards
Parts:
- removed H1, H2: MountingHole, MountingHole:MountingHole_3.2mm_M3_ISO7380_Pad, symbol Mechanical:MountingHole
- added H1, H2: M3, MountingHole:MountingHole_3.2mm_M3_Pad, symbol Mechanical:MountingHole_Pad
- J2: footprint Connector_JST:JST_PH_B4B-PH-SM4-TB_1x04-1MP_P2.00mm_Vertical -> Connector_Molex:Molex_PicoBlade_53398-0471_1x04-1MP_P1.25mm_Vertical
Connections:
- net GND: now also H1.1, H2.1
Changed lines of the file:
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@@
+    (stroke (width 0) (type default))
+  )
+  (wire (pts (xy 130.81 73.66) (xy 128.27 73.66))
     (stroke (width 0) (type default))
   )
@@
   )
   (wire (pts (xy 71.12 69.85) (xy 71.12 77.47))
+    (stroke (width 0) (type default))
+  )
+  (wire (pts (xy 130.81 81.28) (xy 128.27 81.28))
     (stroke (width 0) (type default))
   )
@@
       (effects (font (size 1.27 1.27)) hide)
     )
-    (property "Footprint" "Connector_JST:JST_PH_B4B-PH-SM4-TB_1x04-1MP_P2.00mm_Vertical" (at 118.11 57.15 0)
+    (property "Footprint" "Connector_Molex:Molex_PicoBlade_53398-0471_1x04-1MP_P1.25mm_Vertical" (at 118.11 57.15 0)
       (effects (font (size 1.27 1.27)) hide)
     )
@@
     )
   )
+  (symbol (lib_name "GND_1") (lib_id "power:GND") (at 130.81 81.28 90) (unit 1)
+    (in_bom yes) (on_board yes) (dnp no) (fields_autoplaced)
+    (property "Reference" "#PWR010" (at 137.16 81.28 0)
+      (effects (font (size 1.27 1.27)) hide)
+    )
+    (property "Value" "GND" (at 135.89 81.28 0)
+      (effects (font (size 1.27 1.27)) hide)
+    )
+    (property "Footprint" "" (at 130.81 81.28 0)
+      (effects (font (size 1.27 1.27)) hide)
+    )
+    (property "Datasheet" "" (at 130.81 81.28 0)
+      (effects (font (size 1.27 1.27)) hide)
+    )
+    (pin "1")
+    (instances
+      (project "QRE MiniBoards"
+        (path "/c0d3a82a-eb2a-4d79-a622-f18b88b35157"
+          (reference "#PWR010") (unit 1)
+        )
+      )
+      (project "sumec"
+        (path "/fc70a1a8-ed7c-4a0f-9b1a-f23293528385/cfe10bc0-4e7a-493c-9fb6-0f9ed602f83c"
+          (reference "#PWR016") (unit 1)
+        )
+      )
+    )
+  )
   (symbol (lib_name "GND_1") (lib_id "power:GND") (at 66.04 69.85 0) (unit 1)
     (in_bom yes) (on_board yes) (dnp no) (fields_autoplaced)
@@
     )
   )
-  (symbol (lib_id "Mechanical:MountingHole") (at 121.92 78.74 0) (unit 1)
-    (in_bom yes) (on_board yes) (dnp no)
-    (property "Reference" "H2" (at 116.84 78.74 0)
-      (effects (font (size 1.27 1.27)) (justify left))
-    )
-    (property "Value" "MountingHole" (at 124.46 78.74 0)
-      (effects (font (size 1.27 1.27)) (justify left))
-    )
-    (property "Footprint" "MountingHole:MountingHole_3.2mm_M3_ISO7380_Pad" (at 121.92 78.74 0)
-      (effects (font (size 1.27 1.27)) hide)
-    )
-    (property "Datasheet" "~" (at 121.92 78.74 0)
-      (effects (font (size 1.27 1.27)) hide)
-    )
-    (instances
-      (project "QRE MiniBoards"
-        (path "/c0d3a82a-eb2a-4d79-a622-f18b88b35157"
-          (reference "H2") (unit 1)
+  (symbol (lib_name "GND_1") (lib_id "power:GND") (at 130.81 73.66 90) (unit 1)
+    (in_bom yes) (on_board yes) (dnp no) (fields_autoplaced)
+    (property "Reference" "#PWR09" (at 137.16 73.66 0)
+      (effects (font (size 1.27 1.27)) hide)
+    )
+    (property "Value" "GND" (at 135.89 73.66 0)
+      (effects (font (size 1.27 1.27)) hide)
+    )
+    (property "Footprint" "" (at 130.81 73.66 0)
+      (effects (font (size 1.27 1.27)) hide)
+    )
+    (property "Datasheet" "" (at 130.81 73.66 0)
+      (effects (font (size 1.27 1.27)) hide)
+    )
+    (pin "1")
+    (instances
+      (project "QRE MiniBoards"
+        (path "/c0d3a82a-eb2a-4d79-a622-f18b88b35157"
+          (reference "#PWR09") (unit 1)
+        )
+      )
+      (project "sumec"
+        (path "/fc70a1a8-ed7c-4a0f-9b1a-f23293528385/cfe10bc0-4e7a-493c-9fb6-0f9ed602f83c"
+          (reference "#PWR016") (unit 1)
         )
       )
@@
     )
   )
-  (symbol (lib_id "Mechanical:MountingHole") (at 121.92 71.12 0) (unit 1)
-    (in_bom yes) (on_board yes) (dnp no)
-    (property "Reference" "H1" (at 116.84 71.12 0)
-      (effects (font (size 1.27 1.27)) (justify left))
-    )
-    (property "Value" "MountingHole" (at 124.46 71.12 0)
-      (effects (font (size 1.27 1.27)) (justify left))
-    )
-    (property "Footprint" "MountingHole:MountingHole_3.2mm_M3_ISO7380_Pad" (at 121.92 71.12 0)
-      (effects (font (size 1.27 1.27)) hide)
-    )
-    (property "Datasheet" "~" (at 121.92 71.12 0)
-      (effects (font (size 1.27 1.27)) hide)
-    )
-    (instances
-      (project "QRE MiniBoards"
-        (path "/c0d3a82a-eb2a-4d79-a622-f18b88b35157"
-          (reference "H1") (unit 1)
-        )
-      )
-    )
-  )
   (symbol (lib_id "Device:R") (at 53.34 50.8 180) (unit 1)
     (in_bom yes) (on_board yes) (dnp no)
@@
     )
   )
+  (symbol (lib_id "Mechanical:MountingHole_Pad") (at 125.73 81.28 90) (unit 1)
+    (in_bom yes) (on_board yes) (dnp no)
+    (property "Reference" "H2" (at 120.65 81.28 90)
+      (effects (font (size 1.27 1.27)))
+    )
+    (property "Value" "M3" (at 124.46 77.47 90)
+      (effects (font (size 1.27 1.27)))
+    )
+    (property "Footprint" "MountingHole:MountingHole_3.2mm_M3_Pad" (at 125.73 81.28 0)
+      (effects (font (size 1.27 1.27)) hide)
+    )
+    (property "Datasheet" "~" (at 125.73 81.28 0)
+      (effects (font (size 1.27 1.27)) hide)
+    )
+    (pin "1")
+    (instances
+      (project "QRE MiniBoards"
+        (path "/c0d3a82a-eb2a-4d79-a622-f18b88b35157"
+          (reference "H2") (unit 1)
+        )
+      )
+    )
+  )
   (symbol (lib_name "GND_1") (lib_id "power:GND") (at 66.04 54.61 180) (unit 1)
     (in_bom yes) (on_board yes) (dnp no) (fields_autoplaced)
@@
         )
       )
+    )
+  )
+  (symbol (lib_id "Mechanical:MountingHole_Pad") (at 125.73 73.66 90) (unit 1)
+    (in_bom yes) (on_board yes) (dnp no)
+    (property "Reference" "H1" (at 120.65 73.66 90)
+      (effects (font (size 1.27 1.27)))
+    )
+    (property "Value" "M3" (at 124.46 69.85 90)
+      (effects (font (size 1.27 1.27)))
+    )
+    (property "Footprint" "MountingHole:MountingHole_3.2mm_M3_Pad" (at 125.73 73.66 0)
+      (effects (font (size 1.27 1.27)) hide)
+    )
+    (property "Datasheet" "~" (at 125.73 73.66 0)
+      (effects (font (size 1.27 1.27)) hide)
+    )
+    (pin "1")
+    (instances
+      (project "QRE MiniBoards"
+        (path "/c0d3a82a-eb2a-4d79-a622-f18b88b35157"
+          (reference "H1") (unit 1)
+        )
+      )

Commit message: QRE MiniBoards - update
Parts:
- J2: footprint Connector_Molex:Molex_PicoBlade_53398-0471_1x04-1MP_P1.25mm_Vertical -> Connector_Molex:Molex_PicoBlade_53261-0471_1x04-1MP_P1.25mm_Horizontal
- R1, R2, R3, R4: footprint Resistor_SMD:R_1206_3216Metric_Pad1.30x1.75mm_HandSolder -> Resistor_SMD:R_0805_2012Metric_Pad1.20x1.40mm_HandSolder
- U1, U2: footprint sumec_library:OnSemi_CASE100AQ - QRE1113 -> qre_miniboard_library:OnSemi_CASE100AQ - QRE1113
Connections:
- net QRE1113 A: now also J2.4 (Pin_4); no longer J2.1 (Pin_1)
- net QRE1113 B: now also J2.1 (Pin_1); no longer J2.4 (Pin_4)
Other:
- note added: "Horizontal PicoBlade 4pin connector"
Changed lines of the file:
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@@
     (effects (font (size 3 3) (thickness 0.6) bold (color 0 0 0 1)) (justify left bottom))
+  )
+  (text "Horizontal PicoBlade 4pin connector" (at 102.87 39.37 0)
+    (effects (font (size 1.27 1.27)) (justify left bottom))
   )
   (text "MECHANICAL" (at 113.03 33.02 0)
     (effects (font (size 3 3) (thickness 0.6) bold (color 0 0 0 1)) (justify left bottom))
-  )
-  (global_label "QRE1113 A" (shape input) (at 123.19 54.61 0) (fields_autoplaced)
-    (effects (font (size 0.7 0.7)) (justify left))
-    (property "Intersheetrefs" "${INTERSHEET_REFS}" (at 130.6582 54.61 0)
-      (effects (font (size 1.27 1.27)) (justify left) hide)
-    )
   )
   (global_label "QRE1113 B" (shape input) (at 71.12 73.66 0) (fields_autoplaced)
@@
     )
   )
-  (global_label "QRE1113 B" (shape input) (at 123.19 62.23 0) (fields_autoplaced)
+  (global_label "QRE1113 B" (shape input) (at 123.19 54.61 0) (fields_autoplaced)
     (effects (font (size 0.7 0.7)) (justify left))
-    (property "Intersheetrefs" "${INTERSHEET_REFS}" (at 130.7582 62.23 0)
+    (property "Intersheetrefs" "${INTERSHEET_REFS}" (at 130.7582 54.61 0)
       (effects (font (size 1.27 1.27)) (justify left) hide)
     )
@@
     )
   )
+  (global_label "QRE1113 A" (shape input) (at 123.19 62.23 0) (fields_autoplaced)
+    (effects (font (size 0.7 0.7)) (justify left))
+    (property "Intersheetrefs" "${INTERSHEET_REFS}" (at 130.6582 62.23 0)
+      (effects (font (size 1.27 1.27)) (justify left) hide)
+    )
+  )
   (symbol (lib_id "Connector:Conn_01x04_Pin") (at 118.11 57.15 0) (unit 1)
     (in_bom yes) (on_board yes) (dnp no) (fields_autoplaced)
@@
       (effects (font (size 1.27 1.27)) hide)
     )
-    (property "Footprint" "Connector_Molex:Molex_PicoBlade_53398-0471_1x04-1MP_P1.25mm_Vertical" (at 118.11 57.15 0)
+    (property "Footprint" "Connector_Molex:Molex_PicoBlade_53261-0471_1x04-1MP_P1.25mm_Horizontal" (at 118.11 57.15 0)
       (effects (font (size 1.27 1.27)) hide)
     )
@@
       (effects (font (size 1.27 1.27)) (justify left))
     )
-    (property "Footprint" "sumec_library:OnSemi_CASE100AQ - QRE1113" (at 45.72 62.23 0)
+    (property "Footprint" "qre_miniboard_library:OnSemi_CASE100AQ - QRE1113" (at 45.72 62.23 0)
       (effects (font (size 1.27 1.27)) hide)
     )
@@
       (effects (font (size 1.27 1.27)))
     )
-    (property "Footprint" "Resistor_SMD:R_1206_3216Metric_Pad1.30x1.75mm_HandSolder" (at 72.898 50.8 90)
+    (property "Footprint" "Resistor_SMD:R_0805_2012Metric_Pad1.20x1.40mm_HandSolder" (at 72.898 50.8 90)
       (effects (font (size 1.27 1.27)) hide)
     )
@@
       (effects (font (size 1.27 1.27)))
     )
-    (property "Footprint" "Resistor_SMD:R_1206_3216Metric_Pad1.30x1.75mm_HandSolder" (at 55.118 81.28 90)
+    (property "Footprint" "Resistor_SMD:R_0805_2012Metric_Pad1.20x1.40mm_HandSolder" (at 55.118 81.28 90)
       (effects (font (size 1.27 1.27)) hide)
     )
@@
       (effects (font (size 1.27 1.27)))
     )
-    (property "Footprint" "Resistor_SMD:R_1206_3216Metric_Pad1.30x1.75mm_HandSolder" (at 55.118 50.8 90)
+    (property "Footprint" "Resistor_SMD:R_0805_2012Metric_Pad1.20x1.40mm_HandSolder" (at 55.118 50.8 90)
       (effects (font (size 1.27 1.27)) hide)
     )
@@
       (effects (font (size 1.27 1.27)))
     )
-    (property "Footprint" "Resistor_SMD:R_1206_3216Metric_Pad1.30x1.75mm_HandSolder" (at 72.898 81.28 90)
+    (property "Footprint" "Resistor_SMD:R_0805_2012Metric_Pad1.20x1.40mm_HandSolder" (at 72.898 81.28 90)
       (effects (font (size 1.27 1.27)) hide)
     )
@@
       (effects (font (size 1.27 1.27)) (justify left))
     )
-    (property "Footprint" "sumec_library:OnSemi_CASE100AQ - QRE1113" (at 63.5 62.23 0)
-      (effects (font (size 1.27 1.27)) hide)
-    )
+    (property "Footprint" "qre_miniboard_library:OnSemi_CASE100AQ - QRE1113" (at 63.5 62.23 0)
+      (effects (font (size 1.27 1.27)) hide)
+    )
