File: - PCB -/SUMEC SMD-V2/sumec.kicad_sch (KiCad schematic)
At the start: 3 parts, among them U7 LM1084IS-5.0/NOPB

Commit message: cleanup
Parts:
- removed U7: LM1084IS-5.0/NOPB, Package_TO_SOT_SMD:TO-263-3_TabPin4, symbol Regulator_Linear:LM1084-3.3
- R1: footprint sumec-smd_library:logo even smaller -> (none)
- R2: footprint sumec-smd_library:car cool smol -> (none)
Changed lines of the file:
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@@
     (effects (font (size 5 5) (thickness 1) bold) (justify left bottom) (href "https://www.espressif.com/sites/default/files/documentation/esp32-s3_datasheet_en.pdf"))
-  )
-  (symbol (lib_id "Regulator_Linear:LM1084-3.3") (at 119.38 44.45 0) (unit 1)
-    (in_bom yes) (on_board yes) (dnp no)
-    (property "Reference" "U7" (at 119.38 38.1 0)
-      (effects (font (size 1.27 1.27)))
-    )
-    (property "Value" "LM1084IS-5.0/NOPB" (at 119.38 40.64 0)
-      (effects (font (size 1.27 1.27)))
-    )
-    (property "Footprint" "Package_TO_SOT_SMD:TO-263-3_TabPin4" (at 119.38 38.1 0)
-      (effects (font (size 1.27 1.27) italic) hide)
-    )
-    (property "Datasheet" "http://www.ti.com/lit/ds/symlink/lm1084.pdf" (at 119.38 44.45 0)
-      (effects (font (size 1.27 1.27)) hide)
-    )
-    (pin "1")
-    (pin "2")
-    (pin "3")
-    (instances
-      (project "sumec"
-        (path "/fc70a1a8-ed7c-4a0f-9b1a-f23293528385/2febd48c-c6ec-477b-ac64-6fa98a41fff0"
-          (reference "U7") (unit 1)
-        )
-        (path "/fc70a1a8-ed7c-4a0f-9b1a-f23293528385"
-          (reference "U7") (unit 1)
-        )
-      )
-    )
   )
   (symbol (lib_id "Device:R") (at 153.67 40.64 90) (unit 1)
@@
       (effects (font (size 1.27 1.27)) hide)
     )
-    (property "Footprint" "sumec-smd_library:car cool smol" (at 153.67 42.418 90)
+    (property "Footprint" "" (at 153.67 42.418 90)
       (effects (font (size 1.27 1.27)) hide)
     )
@@
       (effects (font (size 1.27 1.27)) hide)
     )
-    (property "Footprint" "sumec-smd_library:logo even smaller" (at 153.67 38.608 90)
+    (property "Footprint" "" (at 153.67 38.608 90)
       (effects (font (size 1.27 1.27)) hide)
     )

Commit message: sumec SMD V2 schematic update
Parts:
- removed R1, R2: R, symbol Device:R
Connections:
- no-connect marks 4 -> 0
Changed lines of the file:
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@@
     (company "SPŠ NA PROSEKU")
-  )
-  (no_connect (at 129.54 40.64))
-  (no_connect (at 179.07 40.64))
-  (no_connect (at 127 36.83))
-  (no_connect (at 180.34 36.83))
-  (wire (pts (xy 127 36.83) (xy 149.86 36.83))
-    (stroke (width 0) (type default))
-  )
-  (wire (pts (xy 179.07 40.64) (xy 157.48 40.64))
-    (stroke (width 0) (type default))
-  )
-  (wire (pts (xy 180.34 36.83) (xy 157.48 36.83))
-    (stroke (width 0) (type default))
-  )
-  (wire (pts (xy 129.54 40.64) (xy 149.86 40.64))
-    (stroke (width 0) (type default))
   )
   (text "ESP32-S3 Datasheet" (at 115.57 127 0)
     (effects (font (size 5 5) (thickness 1) bold) (justify left bottom) (href "https://www.espressif.com/sites/default/files/documentation/esp32-s3_datasheet_en.pdf"))
-  )
-  (symbol (lib_id "Device:R") (at 153.67 40.64 90) (unit 1)
-    (in_bom yes) (on_board yes) (dnp no) (fields_autoplaced)
-    (property "Reference" "R2" (at 153.67 35.56 90)
-      (effects (font (size 1.27 1.27)) hide)
-    )
-    (property "Value" "R" (at 153.67 38.1 90)
-      (effects (font (size 1.27 1.27)) hide)
-    )
-    (property "Footprint" "" (at 153.67 42.418 90)
-      (effects (font (size 1.27 1.27)) hide)
-    )
-    (property "Datasheet" "~" (at 153.67 40.64 0)
-      (effects (font (size 1.27 1.27)) hide)
-    )
-    (pin "1")
-    (pin "2")
-    (instances
-      (project "sumec"
-        (path "/fc70a1a8-ed7c-4a0f-9b1a-f23293528385"
-          (reference "R2") (unit 1)
-        )
-      )
-    )
   )
   (symbol (lib_id "some magic shit (logo):LOGO") (at 147.32 25.4 0) (unit 1)
@@
         )
       )
-    )
-  )
-  (symbol (lib_id "Device:R") (at 153.67 36.83 90) (unit 1)
-    (in_bom yes) (on_board yes) (dnp no) (fields_autoplaced)
-    (property "Reference" "R1" (at 153.67 31.75 90)
-      (effects (font (size 1.27 1.27)) hide)
-    )
-    (property "Value" "R" (at 153.67 34.29 90)
-      (effects (font (size 1.27 1.27)) hide)
-    )
-    (property "Footprint" "" (at 153.67 38.608 90)
-      (effects (font (size 1.27 1.27)) hide)
-    )
-    (property "Datasheet" "~" (at 153.67 36.83 0)
-      (effects (font (size 1.27 1.27)) hide)
-    )
-    (pin "1")
-    (pin "2")
-    (instances
-      (project "sumec"
-        (path "/fc70a1a8-ed7c-4a0f-9b1a-f23293528385"
-          (reference "R1") (unit 1)
-        )
-      )

Commit message: pcb schematic update
Other:
- note removed: "ESP32-S3 Datasheet"
Changed lines of the file:
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@@
     (company "SPŠ NA PROSEKU")
-  )
-  (text "ESP32-S3 Datasheet" (at 115.57 127 0)
-    (effects (font (size 5 5) (thickness 1) bold) (justify left bottom) (href "https://www.espressif.com/sites/default/files/documentation/esp32-s3_datasheet_en.pdf"))
   )
   (symbol (lib_id "some magic shit (logo):LOGO") (at 147.32 25.4 0) (unit 1)

Commit message: PCB Board Update goodnight hrrrr mimimi
Parts:
- added R3: R, sumec-smdV2_library:R2D2, symbol Device:R
Changed lines of the file:
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@@
     (company "SPŠ NA PROSEKU")
+  )
+  (symbol (lib_id "Device:R") (at 153.67 39.37 90) (unit 1)
+    (in_bom yes) (on_board yes) (dnp no) (fields_autoplaced)
+    (property "Reference" "R3" (at 153.67 34.29 90)
+      (effects (font (size 1.27 1.27)) hide)
+    )
+    (property "Value" "R" (at 153.67 36.83 90)
+      (effects (font (size 1.27 1.27)) hide)
+    )
+    (property "Footprint" "sumec-smdV2_library:R2D2" (at 153.67 41.148 90)
+      (effects (font (size 1.27 1.27)) hide)
+    )
+    (property "Datasheet" "~" (at 153.67 39.37 0)
+      (effects (font (size 1.27 1.27)) hide)
+    )
+    (pin "1")
+    (pin "2")
+    (instances
+      (project "sumec"
+        (path "/fc70a1a8-ed7c-4a0f-9b1a-f23293528385"
+          (reference "R3") (unit 1)
+        )
+      )
+    )
   )
   (symbol (lib_id "some magic shit (logo):LOGO") (at 147.32 25.4 0) (unit 1)

Commit message: PCB - Tracing and component board update
Parts:
- added R8: R, sumec-smdV2_library:Logo, symbol Device:R
Connections:
- no-connect marks 0 -> 4
Changed lines of the file:
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@@
     (company "SPŠ NA PROSEKU")
   )
-  (symbol (lib_id "Device:R") (at 153.67 39.37 90) (unit 1)
+  (no_connect (at 181.61 38.1))
+  (no_connect (at 115.57 34.29))
+  (no_connect (at 115.57 38.1))
+  (no_connect (at 181.61 34.29))
+  (wire (pts (xy 115.57 34.29) (xy 147.32 34.29))
+    (stroke (width 0) (type default))
+  )
+  (wire (pts (xy 115.57 38.1) (xy 147.32 38.1))
+    (stroke (width 0) (type default))
+  )
+  (wire (pts (xy 154.94 38.1) (xy 181.61 38.1))
+    (stroke (width 0) (type default))
+  )
+  (wire (pts (xy 181.61 34.29) (xy 154.94 34.29))
+    (stroke (width 0) (type default))
+  )
+  (symbol (lib_id "Device:R") (at 151.13 34.29 270) (unit 1)
     (in_bom yes) (on_board yes) (dnp no) (fields_autoplaced)
-    (property "Reference" "R3" (at 153.67 34.29 90)
+    (property "Reference" "R3" (at 151.13 39.37 90)
       (effects (font (size 1.27 1.27)) hide)
     )
-    (property "Value" "R" (at 153.67 36.83 90)
+    (property "Value" "R" (at 151.13 36.83 90)
       (effects (font (size 1.27 1.27)) hide)
     )
-    (property "Footprint" "sumec-smdV2_library:R2D2" (at 153.67 41.148 90)
+    (property "Footprint" "sumec-smdV2_library:R2D2" (at 151.13 32.512 90)
       (effects (font (size 1.27 1.27)) hide)
     )
-    (property "Datasheet" "~" (at 153.67 39.37 0)
+    (property "Datasheet" "~" (at 151.13 34.29 0)
       (effects (font (size 1.27 1.27)) hide)
     )
@@
         )
       )
+    )
+  )
+  (symbol (lib_id "Device:R") (at 151.13 38.1 270) (unit 1)
+    (in_bom yes) (on_board yes) (dnp no) (fields_autoplaced)
+    (property "Reference" "R8" (at 151.13 43.18 90)
+      (effects (font (size 1.27 1.27)) hide)
+    )
+    (property "Value" "R" (at 151.13 40.64 90)
+      (effects (font (size 1.27 1.27)) hide)
+    )
+    (property "Footprint" "sumec-smdV2_library:Logo" (at 151.13 36.322 90)
+      (effects (font (size 1.27 1.27)) hide)
+    )
+    (property "Datasheet" "~" (at 151.13 38.1 0)
+      (effects (font (size 1.27 1.27)) hide)
+    )
+    (pin "1")
+    (pin "2")
+    (instances
+      (project "sumec"
+        (path "/fc70a1a8-ed7c-4a0f-9b1a-f23293528385"
+          (reference "R8") (unit 1)
+        )
+      )

Commit message: mateji co jsi kurva delal v slozce PCB??
Changed lines of the file:
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@@
     (in_bom yes) (on_board yes) (dnp no) (fields_autoplaced)
     (property "Reference" "R3" (at 151.13 39.37 90)
-      (effects (font (size 1.27 1.27)) hide)
+      (effects (font (face "Bahnschrift") (size 1.27 1.27)) hide)
     )
     (property "Value" "R" (at 151.13 36.83 90)
-      (effects (font (size 1.27 1.27)) hide)
+      (effects (font (face "Bahnschrift") (size 1.27 1.27)) hide)
     )
     (property "Footprint" "sumec-smdV2_library:R2D2" (at 151.13 32.512 90)
-      (effects (font (size 1.27 1.27)) hide)
+      (effects (font (face "Bahnschrift") (size 1.27 1.27)) hide)
     )
     (property "Datasheet" "~" (at 151.13 34.29 0)
-      (effects (font (size 1.27 1.27)) hide)
+      (effects (font (face "Bahnschrift") (size 1.27 1.27)) hide)
     )
     (pin "1")
@@
     (in_bom yes) (on_board yes) (dnp no) (fields_autoplaced)
     (property "Reference" "R8" (at 151.13 43.18 90)
-      (effects (font (size 1.27 1.27)) hide)
+      (effects (font (face "Bahnschrift") (size 1.27 1.27)) hide)
     )
     (property "Value" "R" (at 151.13 40.64 90)
-      (effects (font (size 1.27 1.27)) hide)
+      (effects (font (face "Bahnschrift") (size 1.27 1.27)) hide)
     )
     (property "Footprint" "sumec-smdV2_library:Logo" (at 151.13 36.322 90)
-      (effects (font (size 1.27 1.27)) hide)
+      (effects (font (face "Bahnschrift") (size 1.27 1.27)) hide)
     )
     (property "Datasheet" "~" (at 151.13 38.1 0)
-      (effects (font (size 1.27 1.27)) hide)
+      (effects (font (face "Bahnschrift") (size 1.27 1.27)) hide)
     )
     (pin "1")
@@
     (in_bom yes) (on_board yes) (dnp no) (fields_autoplaced)
     (property "Reference" "#G1" (at 147.32 14.7743 0)
-      (effects (font (size 1.27 1.27)) hide)
+      (effects (font (face "Bahnschrift") (size 1.27 1.27)) hide)
     )
     (property "Value" "LOGO" (at 147.32 36.0257 0)
-      (effects (font (size 1.27 1.27)) hide)
+      (effects (font (face "Bahnschrift") (size 1.27 1.27)) hide)
     )
     (property "Footprint" "" (at 147.32 25.4 0)
-      (effects (font (size 1.27 1.27)) hide)
+      (effects (font (face "Bahnschrift") (size 1.27 1.27)) hide)
     )
     (property "Datasheet" "" (at 147.32 25.4 0)
-      (effects (font (size 1.27 1.27)) hide)
+      (effects (font (face "Bahnschrift") (size 1.27 1.27)) hide)
     )
     (instances
@@
     (stroke (width 0.1524) (type solid) (color 0 0 0 1))
     (fill (color 255 255 255 1.0000))
-    (property "Sheetname" "MECHANICS" (at 39.37 133.35 0)
-      (effects (font (size 5 5) bold (color 0 0 0 1)) (justify left bottom))
+    (property "Sheetname" "MECHANICS" (at 44.45 133.35 0)
+      (effects (font (face "Bahnschrift") (size 5 5) bold (color 0 0 0 1)) (justify left bottom))
     )
     (property "Sheetfile" "MECHANICS.kicad_sch" (at 27.94 154.94 0)
-      (effects (font (size 1.27 1.27) (color 0 0 0 1)) (justify left top))
+      (effects (font (face "Bahnschrift") (size 1.27 1.27) (color 0 0 0 1)) (justify left top))
     )
     (instances
@@
     (stroke (width 0.1524) (type solid) (color 0 0 0 1))
     (fill (color 255 255 255 1.0000))
-    (property "Sheetname" "MCU" (at 53.34 73.66 0)
-      (effects (font (size 5 5) bold (color 0 0 0 1)) (justify left bottom))
+    (property "Sheetname" "MCU" (at 55.88 73.66 0)
+      (effects (font (face "Bahnschrift") (size 5 5) bold (color 0 0 0 1)) (justify left bottom))
     )
     (property "Sheetfile" "MCU.kicad_sch" (at 27.94 96.52 0)
-      (effects (font (size 1.27 1.27) (color 0 0 0 1)) (justify left top))
+      (effects (font (face "Bahnschrift") (size 1.27 1.27) (color 0 0 0 1)) (justify left top))
     )
     (instances
@@
     (stroke (width 0.1524) (type solid) (color 0 0 0 1))
     (fill (color 255 255 255 1.0000))
-    (property "Sheetname" "POWER SUPPLY" (at 209.55 73.66 0)
-      (effects (font (size 5 5) bold (color 0 0 0 1)) (justify left bottom))
+    (property "Sheetname" "POWER SUPPLY" (at 214.63 74.93 0)
+      (effects (font (face "Bahnschrift") (size 5 5) bold (color 0 0 0 1)) (justify left bottom))
     )
     (property "Sheetfile" "POWER SUPPLY.kicad_sch" (at 204.47 96.52 0)
-      (effects (font (size 1.27 1.27) (color 0 0 0 1)) (justify left top))
+      (effects (font (face "Bahnschrift") (size 1.27 1.27) (color 0 0 0 1)) (justify left top))
     )
     (instances
@@
     (fill (color 255 255 255 1.0000))
     (property "Sheetname" "SENSORS" (at 133.35 73.66 0)
-      (effects (font (size 5 5) bold (color 0 0 0 1)) (justify left bottom))
+      (effects (font (face "Bahnschrift") (size 5 5) bold (color 0 0 0 1)) (justify left bottom))
     )
     (property "Sheetfile" "SENSORS.kicad_sch" (at 115.57 95.8346 0)
-      (effects (font (size 1.27 1.27) (color 0 0 0 1)) (justify left top))
+      (effects (font (face "Bahnschrift") (size 1.27 1.27) (color 0 0 0 1)) (justify left top))
     )
     (property "Field2" "" (at 115.57 48.26 0)
-      (effects (font (size 1.27 1.27)) hide)
+      (effects (font (face "Bahnschrift") (size 1.27 1.27)) hide)
     )
     (instances
