File: - PCB -/SUMEC SMD-V2 (revert)/MCU.kicad_sch (KiCad schematic)
At the start: 29 parts, among them IC2 DRV8874PWPR, IC3 DRV8874PWPR, J5 TYPE-C-31-M-12, SW2 SW_Push, SW3 SW_Push, U2 ESP32-S3-WROOM-1, U3 USBLC6-2SC6

Commit message: fuckup reverted???
Parts:
- gave numbers to parts that had none: 9
- renumbered C12 to C16, C12 to C3, C12 to C5
