File: - PCB -/SUMEC SMD-V2 (revert)/MECHANICS.kicad_sch (KiCad schematic)
At the start: 7 parts, among them J1 Conn_01x04_Pin, SW1 SW_Push, SW4 SW_DPDT_x2

Commit message: fuckup reverted???
Parts:
- gave numbers to parts that had none: 1
Changed lines of the file:
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@@
           (reference "J1") (unit 1)
-        )
-        (path "/fc70a1a8-ed7c-4a0f-9b1a-f23293528385/2febd48c-c6ec-477b-ac64-6fa98a41fff0"
-          (reference "J?") (unit 1)
         )
       )
@@
   (symbol (lib_id "Connector:Conn_01x01_Pin") (at 168.91 128.27 0) (unit 1)
     (in_bom yes) (on_board yes) (dnp no)
-    (property "Reference" "J?" (at 166.37 128.27 0)
+    (property "Reference" "J2" (at 166.37 128.27 0)
       (effects (font (size 1.27 1.27)))
     )
@@
     (instances
       (project "sumec"
-        (path "/fc70a1a8-ed7c-4a0f-9b1a-f23293528385/11aa20d4-c4ff-49be-9179-c2911da50f67"
-          (reference "J?") (unit 1)
-        )
         (path "/fc70a1a8-ed7c-4a0f-9b1a-f23293528385/05a35bad-c108-46ad-8f95-76319a60a14f"
           (reference "J2") (unit 1)
