File: - PCB -/SUMEC SMD-V2 (revert)/SENSORS.kicad_sch (KiCad schematic)
At the start: 12 parts, among them J10 Conn_01x03_Pin, J3 Conn_01x04_Pin, J4 Conn_01x03_Pin, J9 Conn_01x03_Pin

Commit message: fuckup reverted???
Parts:
- gave numbers to parts that had none: 4
- renumbered C12 to C14, C12 to C15
Other:
- note added: "When pin 5 is connected to ground, TF-Luna enters I2C mode, then its pin 2 is used as SDA data and pin 3 is the SCL clock sending data. Addresses are saved using Nat Simak's program."
- note removed: "When pin 5 is connected to ground, TF-Luna enters I2C mode, then its pin 2 is used as SDA data and pin 3 is the SCL clock sending data. Addresses are saved using Mr_Simak program."
