File: - PCB -/SUMEC SMD-V2 (revert)/sumec.kicad_pcb (KiCad board)
At the start: 2 copper layers, 95 x 55 mm, 57 parts, among them IC2 DRV8874PWPR, IC3 DRV8874PWPR, J1 Conn_01x04_Pin, J10 Conn_01x03_Pin, J11 XT30PW-M, J2 Conn_01x01_Pin, J3 Conn_01x04_Pin, J4 Conn_01x03_Pin, J5 TYPE-C-31-M-12, J6 Conn_01x06_Pin, J7 Conn_01x06_Pin, J8 Conn_01x06_Pin, J9 Conn_01x03_Pin, SW1 SW_Push, SW2 SW_Push, SW3 SW_Push, SW4 SW_DPDT_x2, U1 LM1084-3.3, U2 ESP32-S3-WROOM-1, U3 USBLC6-2SC6, U4 LM1084-5.0, U5 TSOP382xx

Commit message: fuckup reverted???
Parts:
- moved J11 8.50 mm to (161.2, 122.2)
- moved C15 3.98 mm to (146.8, 111.5)
- moved J10 3.98 mm to (151.5, 111.5)
Routing:
- net VBATT: track 7.50 -> 12.9 mm
- net +3V3: track 220.0 -> 216.3 mm
- net +12V: track 74.7 -> 75.7 mm
- net SHARP 2: track 62.4 -> 63.2 mm
