File: - PCB -/RC-5 Remote Controler/RC-5 Remote Controler.kicad_pcb (KiCad board)
At the start: 2 copper layers, 40 x 59.8 mm, 11 parts, among them SW1 SW_Push, SW2 SW_Push, SW3 SW_Push, SW4 SW_Push

Commit message: PCB RC5 update
Routing:
- net GND: track 63.7 -> 1.38 mm, vias 2 -> 3
- net Net-(A1-D5): track 38.9 -> 39.4 mm
- added copper zone on B.Cu, net GND
