File: - PCB -/Remote/Remote.kicad_sch (KiCad schematic)
At the start: 48 parts

Commit message: Updated schematic
Parts:
- added J?: Conn_01x02_Pin, symbol Connector:Conn_01x02_Pin
Connections:
- net +3V0: now also J?.1 (Pin_1)
- net GND: now also J?.2 (Pin_2)
Other:
- note added: "IR_LEDS"
- note added: "MCU"
- note added: "POWER_SUPP"
- note added: "PROG"
- note added: "START_STOP"
- note added: "SWITCHES"
- note added: "S_LEDS"
- note added: "proc jako pullupy se tady pouzivaji 4.7k? na co je crystal oscilator? na co jsou 2.2R? proc decouple kondenzaotry maji stejnou hodnotu? proc nekteri kondenzatory maji 18pF? na co je nmos?"
- note removed: "Prog"
- note removed: "Start/Stop"
- note removed: "proc jako pullupy se tady pouzivaji 4.7k? na co je crystal oscilator? na co jsou 2.2R? proc decouple kondenzaotry maji stejnou hodnotu? proc nekteri kondenzatory maji 18pF?"
- company: (none) -> SPŠ NA PROSEKU
- title: (none) -> RC5_Remote_Starter
- moved on the sheet: BT?, C?, D?, J?, Q?, R?, SW?, U?, Y?

Commit message: PCB schematic update
Parts:
- C1, C3, C4, C6: renamed from C?; footprint (none) -> Capacitor_SMD:C_0805_2012Metric_Pad1.18x1.45mm_HandSolder
- C2, C5: renamed from C?; footprint (none) -> Capacitor_Tantalum_SMD:CP_EIA-3216-18_Kemet-A_Pad1.58x1.35mm_HandSolder
- D1, D2, D3, D4: renamed from D?; footprint LED_THT:LED_D3.0mm_IRBlack -> LED_THT:LED_D3.0mm_Horizontal_O3.81mm_Z10.0mm
- D5, D6, D7, D8: renamed from D?; footprint (none) -> LED_SMD:LED_0805_2012Metric_Pad1.15x1.40mm_HandSolder
- J1, J2, J3, J5: renamed from J?; footprint (none) -> Connector_PinHeader_2.54mm:PinHeader_1x02_P2.54mm_Vertical
- J4: renamed from J?; footprint (none) -> Connector_PinHeader_2.54mm:PinHeader_2x03_P2.54mm_Vertical
- Q1: renamed from Q?; footprint (none) -> Package_TO_SOT_SMD:TSOT-23_HandSoldering
- R1, R10, R11, R12, R13, R14, R15, R16, R17, R19, R2, R20, R21, R22, R3, R4, R5, R6, R7, R8, R9: renamed from R?; footprint (none) -> Resistor_SMD:R_0805_2012Metric_Pad1.20x1.40mm_HandSolder
- SW1, SW2, SW3: renamed from SW?; footprint (none) -> Button_Switch_THT:SW_PUSH_6mm
- SW4: renamed from SW?; footprint (none) -> Button_Switch_THT:SW_DIP_SPSTx05_Slide_9.78x14.88mm_W7.62mm_P2.54mm
- Y1: renamed from Y?; footprint (none) -> sumec-remote_library:crystal_footprint
- gave numbers to parts that had none: 3
Other:
- note added: "CONNECTORS"
- moved on the sheet: D1, D2, D3, R6, R7, R8

Commit message: Update Remote.kicad_sch
Other:
- note added: "ABL-16.000MHZ-B2 C_{LOAD} = 18 pF"
- note added: "DMG6968U-7 R_{DS(ON)} = 23 Ohm"
- note added: "IR204-A I_{F} = 100 mA V_{F} = 1.4 V"
- note added: "TSUS5400 I_{F} = 100 mA V_{F} = 1.7 V R_{IR} = (V_{SUPP}-V_{F})/I_{F} = = (3-1.7)/0.1 = 13 Ohm for t_{p} < 100 us I_{F} = 1.5 A V_{F} = 2.2 V R_{IR} = (V_{SUPP}-V_{F})/I_{F} = = (3-2.2)/1.5 = 0.53 Ohm"
Changed lines of the file:
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@@
+		)
+	)
+	(text "IR204-A\nI_{F} = 100 mA\nV_{F} = 1.4 V"
+		(exclude_from_sim no)
+		(at 118.872 89.662 0)
+		(effects
+			(font
+				(size 1.27 1.27)
+			)
+			(justify left top)
 		)
 	)
@@
 		)
 	)
+	(text "TSUS5400\nI_{F} = 100 mA\nV_{F} = 1.7 V\n\nR_{IR} = (V_{SUPP}-V_{F})/I_{F} =\n= (3-1.7)/0.1 = 13 Ohm\n\nfor t_{p} < 100 us\nI_{F} = 1.5 A\nV_{F} = 2.2 V\n\nR_{IR} = (V_{SUPP}-V_{F})/I_{F} =\n= (3-2.2)/1.5 = 0.53 Ohm\n"
+		(exclude_from_sim no)
+		(at 118.872 52.832 0)
+		(effects
+			(font
+				(size 1.27 1.27)
+			)
+			(justify left top)
+		)
+	)
 	(text "S_LEDS"
 		(exclude_from_sim no)
@@
 				(color 0 0 0 1)
 			)
+		)
+	)
+	(text "ABL-16.000MHZ-B2\nC_{LOAD} = 18 pF"
+		(exclude_from_sim no)
+		(at 263.398 76.708 0)
+		(effects
+			(font
+				(size 1.27 1.27)
+			)
+			(justify left top)
+			(href "https://cz.mouser.com/datasheet/2/3/ABL-1774766.pdf")
 		)
 	)
@@
 		)
 	)
+	(text "DMG6968U-7\nR_{DS(ON)} = 23 Ohm"
+		(exclude_from_sim no)
+		(at 79.502 126.238 0)
+		(effects
+			(font
+				(size 1.27 1.27)
+			)
+			(justify left top)
+		)
+	)

Commit message: pcb remote update
Parts:
- removed R18: 4k7, Resistor_SMD:R_0805_2012Metric_Pad1.20x1.40mm_HandSolder, symbol remote_V0_04_-eagle-import:R-EU_R0805WP
- added R18: 10k, Resistor_SMD:R_0805_2012Metric_Pad1.20x1.40mm_HandSolder, symbol Device:R
- BT1: footprint Battery:BatteryHolder_Keystone_2462_2xAA -> Battery:BatteryHolder_Keystone_2462_2xAA - no holes
- R1, R13, R14, R15, R16, R17, R2, R3, R5: value 4.7k -> 10k
Connections:
- net +3V0: now also R18.2
- net ADDR0: now also R14.2; no longer R13.2
- net ADDR1: no longer R14.2
- net GND: now also R5.1; no longer R5.2
- net RESET: now also R18.1
- net SW_PROG: now also R3.1; no longer R3.2
- net SW_START: now also R1.1; no longer R1.2
- net SW_STOP: now also R2.1; no longer R2.2
- net at SW2.1: now also R2.2; no longer R2.1
- net at SW3.1: now also R3.2; no longer R3.1
- net at Q1.2 (G), R4.2: now also R5.2; no longer R5.1
- net at SW1.1: now also R1.2; no longer R1.1
- net at SW4.10: now also R14.1; no longer R13.1
- net at SW4.9: no longer R14.1
Other:
- note removed: "hm?"
- note removed: "proc jako pullupy se tady pouzivaji 4.7k? na co je crystal oscilator? na co jsou 2.2R? proc decouple kondenzaotry maji stejnou hodnotu? proc nekteri kondenzatory maji 18pF? na co je nmos?"

Commit message: remote pcb
Parts:
- removed J1, J2, J3, J5: Conn_01x02_Pin, Connector_PinHeader_2.54mm:PinHeader_1x02_P2.54mm_Vertical, symbol Connector:Conn_01x02_Pin
- removed R10, R11: 2.2R, Resistor_SMD:R_0805_2012Metric_Pad1.20x1.40mm_HandSolder, symbol Device:R
- R9: value 2.2R -> R; footprint Resistor_SMD:R_0805_2012Metric_Pad1.20x1.40mm_HandSolder -> sumec-remote_library:purosidenegative
Connections:
- net ADDR1: now also R13.2
- net at Q1.1 (D), R6.1, R7.1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: no longer R9.1
- net at SW4.9: now also R13.1
- no-connect marks 7 -> 9
Other:
- note added: "MISC"
- moved on the sheet: BT1, C1, C2, C3, C4, C5, C6, D1, D2, D3, D4, D5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

Commit message: remote controller rebuild
Parts:
- removed R13, R14, R15, R16, R17: 10k, Resistor_SMD:R_0805_2012Metric_Pad1.20x1.40mm_HandSolder, symbol Device:R
- removed SW4: SW_DIP_x05, Button_Switch_THT:SW_DIP_SPSTx05_Slide_9.78x14.88mm_W7.62mm_P2.54mm, symbol Switch:SW_DIP_x05
- removed Y1: Crystal, sumec-remote_library:crystal_footprint, symbol Device:Crystal
- added IC1: DS04-254-1-05BK-SMT, SUMEC:DS04254105BKSMT, symbol SUMEC:DS04-254-1-05BK-SMT
- added RN1: YC248-JR-0710KL, SUMEC:YC248JR0710KL, symbol SUMEC:YC248-JR-0710KL
- added Y1: ABM8G-16.000MHZ-18-D2Y-T, SUMEC:ABM8G, symbol SUMEC:ABM8G-16.000MHZ-18-D2Y-T
- Q1: value NMOS -> DMG6968U-7
Connections:
- net ADDR0: now also RN1.5
- net ADDR1: now also RN1.4
- net ADDR2: now also RN1.3
- net ADDR3: now also RN1.2
- net ADDR4: now also RN1.1
- net GND: now also C3.1, C4.1, IC1.1 (COM_1), IC1.3 (COM_2), IC1.5 (COM_3), IC1.7 (COM_4), IC1.9 (COM_5), Y1.2 (GND_1), Y1.4 (GND_2); no longer C3.2, C4.2
- net XTAL1: now reaches U1.7 (XTAL1/PB6)
- net XTAL1: now also C3.2, Y1.1 (XTAL_1); no longer C3.1
- net XTAL2: now reaches U1.8 (XTAL2/PB7)
- net XTAL2: now also C4.2, Y1.3 (XTAL_2); no longer C4.1
- new net: IC1.10 (NO_5), RN1.12
- new net: IC1.8 (NO_4), RN1.13
- new net: IC1.6 (NO_3), RN1.14
- new net: IC1.4 (NO_2), RN1.15
- new net: IC1.2 (NO_1), RN1.16
Other:
- note added: "DMG6968U-7 R_{DS(ON)} = 23 mOhm"
- note removed: "ABL-16.000MHZ-B2 C_{LOAD} = 18 pF"
- note removed: "DMG6968U-7 R_{DS(ON)} = 23 Ohm"
- note removed: "START_STOP"
- moved on the sheet: C1, C2, C3, C4, D1, D2, D3, D4, R12, R18, R4, R5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

Commit message: Remote PCB , rebuild update
Parts:
- added H1, H2, H3, H4: Mounting Hole M3, MountingHole:MountingHole_3.2mm_M3_ISO7380_Pad, symbol Mechanical:MountingHole_Pad
- added R16: R, sumec-remote_library:nerd, symbol Device:R
- added R17: R, sumec-remote_library:boi, symbol Device:R
- IC1: footprint SUMEC:DS04254105BKSMT -> sumec-remote_library:dip_switch
- RN1: footprint SUMEC:YC248JR0710KL -> sumec-remote_library:resistor_array
- Y1: footprint SUMEC:ABM8G -> sumec-remote_library:crystal_smd
- renumbered C5 to C1, C6 to C2, C1 to C3, C2 to C4, C3 to C5, C4 to C6, J4 to J1, R4 to R1, R19 to R10, R20 to R11, R21 to R12, R22 to R13, R9 to R14, R18 to R15, R6 to R2, R5 to R3, R7 to R4, R1 to R5, R2 to R6, R3 to R7, R12 to R9
Connections:
- net GND: now also H1.1, H2.1, H3.1, H4.1
- no-connect marks 9 -> 19
Other:
- note added: "RESISTOR ARRAY"
- moved on the sheet: BT1, C1, C2, C3, C4, C5, C6, D1, D2, D3, D4, D5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

Commit message: PCB edit
Parts:
- removed H1, H2: Mounting Hole M3, MountingHole:MountingHole_3.2mm_M3_ISO7380_Pad, symbol Mechanical:MountingHole_Pad
Changed lines of the file:
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@@
-	)
-	(symbol
-		(lib_id "Mechanical:MountingHole_Pad")
-		(at 289.56 290.83 90)
-		(unit 1)
-		(exclude_from_sim yes)
-		(in_bom no)
-		(on_board yes)
-		(dnp no)
-		(fields_autoplaced yes)
-		(property "Reference" "H2"
-			(at 288.29 284.48 90)
-			(effects
-				(font
-					(size 1.27 1.27)
-				)
-			)
-		)
-		(property "Value" "Mounting Hole M3"
-			(at 288.29 287.02 90)
-			(effects
-				(font
-					(size 1.27 1.27)
-				)
-			)
-		)
-		(property "Footprint" "MountingHole:MountingHole_3.2mm_M3_ISO7380_Pad"
-			(at 289.56 290.83 0)
-			(effects
-				(font
-					(size 1.27 1.27)
-				)
-				(hide yes)
-			)
-		)
-		(property "Datasheet" "~"
-			(at 289.56 290.83 0)
-			(effects
-				(font
-					(size 1.27 1.27)
-				)
-				(hide yes)
-			)
-		)
-		(property "Description" "Mounting Hole with connection"
-			(at 289.56 290.83 0)
-			(effects
-				(font
-					(size 1.27 1.27)
-				)
-				(hide yes)
-			)
-		)
-		(pin "1"
-		)
-		(instances
-			(project "Remote"
-				(path "/d5f3a3bc-154f-419d-b1e3-9310b24e53c3"
-					(reference "H2")
-					(unit 1)
-				)
-			)
-		)
 	)
 	(symbol
@@
 					(unit 1)
 				)
-			)
-		)
-	)
-	(symbol
-		(lib_id "Mechanical:MountingHole_Pad")
-		(at 289.56 313.69 90)
-		(unit 1)
-		(exclude_from_sim yes)
-		(in_bom no)
-		(on_board yes)
-		(dnp no)
-		(fields_autoplaced yes)
-		(property "Reference" "H1"
-			(at 288.29 307.34 90)
-			(effects
-				(font
-					(size 1.27 1.27)
-				)
-			)
-		)
-		(property "Value" "Mounting Hole M3"
-			(at 288.29 309.88 90)
-			(effects
-				(font
-					(size 1.27 1.27)
-				)
-			)
-		)
-		(property "Footprint" "MountingHole:MountingHole_3.2mm_M3_ISO7380_Pad"
-			(at 289.56 313.69 0)
-			(effects
-				(font
-					(size 1.27 1.27)
-				)
-				(hide yes)
-			)
-		)
-		(property "Datasheet" "~"
-			(at 289.56 313.69 0)
-			(effects
-				(font
-					(size 1.27 1.27)
-				)
-				(hide yes)
-			)
-		)
-		(property "Description" "Mounting Hole with connection"
-			(at 289.56 313.69 0)
-			(effects
-				(font
-					(size 1.27 1.27)
-				)
-				(hide yes)
-			)
-		)
-		(pin "1"
-		)
-		(instances
-			(project "Remote"
-				(path "/d5f3a3bc-154f-419d-b1e3-9310b24e53c3"
-					(reference "H1")
-					(unit 1)
-				)
