File: -PCB-/SUMEC_MK_IV/SENSORS.kicad_sch (KiCad schematic)
At the start: 15 parts, among them J10 Conn_01x04_Pin, J11 Conn_01x03_Pin, J2 Conn_01x03_Pin, J3 Conn_01x06_Pin, J4 Conn_01x06_Pin, J5 Conn_01x03_Pin, J6 Conn_01x06_Pin, J7 Conn_01x03_Pin, J8 Conn_01x03_Pin, J9 Conn_01x03_Pin, U3 TSOP382xx

Commit message: Footprints added
Parts:
- J7, J8, J9: footprint (none) -> Connector_Molex:Molex_PicoBlade_53398-0371_1x03-1MP_P1.25mm_Vertical
Changed lines of the file:
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@@
 		(on_board yes)
 		(dnp no)
-		(property "Reference" "#PWR059"
+		(property "Reference" "#PWR064"
 			(at 256.54 64.77 0)
 			(effects
@@
 			(project "SUMEC_MK_IV"
 				(path "/900bd7ac-cdf9-4a2f-8b1f-2c21e3760046/a4783534-f11a-41d1-a455-2e16f5dc258a"
-					(reference "#PWR059")
+					(reference "#PWR064")
 					(unit 1)
 				)
@@
 		(on_board yes)
 		(dnp no)
-		(property "Reference" "#PWR050"
+		(property "Reference" "#PWR055"
 			(at 227.33 106.68 0)
 			(effects
@@
 			(project "SUMEC_MK_IV"
 				(path "/900bd7ac-cdf9-4a2f-8b1f-2c21e3760046/a4783534-f11a-41d1-a455-2e16f5dc258a"
-					(reference "#PWR050")
+					(reference "#PWR055")
 					(unit 1)
 				)
@@
 		(dnp no)
 		(fields_autoplaced yes)
-		(property "Reference" "#PWR041"
+		(property "Reference" "#PWR046"
 			(at 63.5 121.92 0)
 			(effects
@@
 			(project "SUMEC_MK_IV"
 				(path "/900bd7ac-cdf9-4a2f-8b1f-2c21e3760046/a4783534-f11a-41d1-a455-2e16f5dc258a"
-					(reference "#PWR041")
+					(reference "#PWR046")
 					(unit 1)
 				)
@@
 		(on_board yes)
 		(dnp no)
-		(property "Reference" "#PWR040"
+		(property "Reference" "#PWR045"
 			(at 52.07 114.3 0)
 			(effects
@@
 			(project "SUMEC_MK_IV"
 				(path "/900bd7ac-cdf9-4a2f-8b1f-2c21e3760046/a4783534-f11a-41d1-a455-2e16f5dc258a"
-					(reference "#PWR040")
+					(reference "#PWR045")
 					(unit 1)
 				)
@@
 		(on_board yes)
 		(dnp no)
-		(property "Reference" "#PWR046"
+		(property "Reference" "#PWR051"
 			(at 105.41 168.91 0)
 			(effects
@@
 			(project "SUMEC_MK_IV"
 				(path "/900bd7ac-cdf9-4a2f-8b1f-2c21e3760046/a4783534-f11a-41d1-a455-2e16f5dc258a"
-					(reference "#PWR046")
+					(reference "#PWR051")
 					(unit 1)
 				)
@@
 		(on_board yes)
 		(dnp no)
-		(property "Reference" "#PWR042"
+		(property "Reference" "#PWR047"
 			(at 71.12 168.91 0)
 			(effects
@@
 			(project "SUMEC_MK_IV"
 				(path "/900bd7ac-cdf9-4a2f-8b1f-2c21e3760046/a4783534-f11a-41d1-a455-2e16f5dc258a"
-					(reference "#PWR042")
+					(reference "#PWR047")
 					(unit 1)
 				)
@@
 		(on_board yes)
 		(dnp no)
-		(property "Reference" "#PWR038"
+		(property "Reference" "#PWR043"
 			(at 31.75 114.3 0)
 			(effects
@@
 			(project "SUMEC_MK_IV"
 				(path "/900bd7ac-cdf9-4a2f-8b1f-2c21e3760046/a4783534-f11a-41d1-a455-2e16f5dc258a"
-					(reference "#PWR038")
+					(reference "#PWR043")
 					(unit 1)
 				)
@@
 			)
 		)
-		(property "Footprint" ""
+		(property "Footprint" "Connector_Molex:Molex_PicoBlade_53398-0371_1x03-1MP_P1.25mm_Vertical"
 			(at 233.68 111.76 0)
 			(effects
@@
 		(on_board yes)
 		(dnp no)
-		(property "Reference" "#PWR047"
+		(property "Reference" "#PWR052"
 			(at 96.52 66.04 0)
 			(effects
@@
 			(project "SUMEC_MK_IV"
 				(path "/900bd7ac-cdf9-4a2f-8b1f-2c21e3760046/a4783534-f11a-41d1-a455-2e16f5dc258a"
-					(reference "#PWR047")
+					(reference "#PWR052")
 					(unit 1)
 				)
@@
 		(dnp no)
 		(fields_autoplaced yes)
-		(property "Reference" "#PWR052"
+		(property "Reference" "#PWR057"
 			(at 251.46 67.31 0)
 			(effects
@@
 			(project "SUMEC_MK_IV"
 				(path "/900bd7ac-cdf9-4a2f-8b1f-2c21e3760046/a4783534-f11a-41d1-a455-2e16f5dc258a"
-					(reference "#PWR052")
+					(reference "#PWR057")
 					(unit 1)
 				)
@@
 		(on_board yes)
 		(dnp no)
-		(property "Reference" "#PWR043"
+		(property "Reference" "#PWR048"
 			(at 62.23 161.29 0)
 			(effects
@@
 			(project "SUMEC_MK_IV"
 				(path "/900bd7ac-cdf9-4a2f-8b1f-2c21e3760046/a4783534-f11a-41d1-a455-2e16f5dc258a"
-					(reference "#PWR043")
+					(reference "#PWR048")
 					(unit 1)
 				)
@@
 		(dnp no)
 		(fields_autoplaced yes)
-		(property "Reference" "#PWR049"
+		(property "Reference" "#PWR054"
 			(at 107.95 60.96 0)
 			(effects
@@
 			(project "SUMEC_MK_IV"
 				(path "/900bd7ac-cdf9-4a2f-8b1f-2c21e3760046/a4783534-f11a-41d1-a455-2e16f5dc258a"
-					(reference "#PWR049")
+					(reference "#PWR054")
 					(unit 1)
 				)
@@
 		(on_board yes)
 		(dnp no)
-		(property "Reference" "#PWR054"
+		(property "Reference" "#PWR059"
 			(at 245.11 48.26 0)
 			(effects
@@
 			(project "SUMEC_MK_IV"
 				(path "/900bd7ac-cdf9-4a2f-8b1f-2c21e3760046/a4783534-f11a-41d1-a455-2e16f5dc258a"
-					(reference "#PWR054")
+					(reference "#PWR059")
 					(unit 1)
 				)
@@
 		(on_board yes)
 		(dnp no)
-		(property "Reference" "#PWR051"
+		(property "Reference" "#PWR056"
 			(at 219.71 104.14 0)
 			(effects
@@
 			(project "SUMEC_MK_IV"
 				(path "/900bd7ac-cdf9-4a2f-8b1f-2c21e3760046/a4783534-f11a-41d1-a455-2e16f5dc258a"
-					(reference "#PWR051")
+					(reference "#PWR056")
 					(unit 1)
 				)
@@
 		(dnp no)
 		(fields_autoplaced yes)
-		(property "Reference" "#PWR053"
+		(property "Reference" "#PWR058"
 			(at 254 45.72 0)
 			(effects
@@
 			(project "SUMEC_MK_IV"
 				(path "/900bd7ac-cdf9-4a2f-8b1f-2c21e3760046/a4783534-f11a-41d1-a455-2e16f5dc258a"
-					(reference "#PWR053")
+					(reference "#PWR058")
 					(unit 1)
 				)
@@
 		(on_board yes)
 		(dnp no)
-		(property "Reference" "#PWR057"
+		(property "Reference" "#PWR062"
 			(at 247.65 97.79 0)
 			(effects
@@
 			(project "SUMEC_MK_IV"
 				(path "/900bd7ac-cdf9-4a2f-8b1f-2c21e3760046/a4783534-f11a-41d1-a455-2e16f5dc258a"
-					(reference "#PWR057")
+					(reference "#PWR062")
 					(unit 1)
 				)
@@
 		(on_board yes)
 		(dnp no)
-		(property "Reference" "#PWR055"
+		(property "Reference" "#PWR060"
 			(at 255.27 100.33 0)
 			(effects
@@
 			(project "SUMEC_MK_IV"
 				(path "/900bd7ac-cdf9-4a2f-8b1f-2c21e3760046/a4783534-f11a-41d1-a455-2e16f5dc258a"
-					(reference "#PWR055")
+					(reference "#PWR060")
 					(unit 1)
 				)
@@
 			)
 		)
-		(property "Footprint" ""
+		(property "Footprint" "Connector_Molex:Molex_PicoBlade_53398-0371_1x03-1MP_P1.25mm_Vertical"
 			(at 233.68 97.79 0)
 			(effects
@@
 		(dnp no)
 		(fields_autoplaced yes)
-		(property "Reference" "#PWR039"
+		(property "Reference" "#PWR044"
 			(at 43.18 121.92 0)
 			(effects
@@
 			(project "SUMEC_MK_IV"
 				(path "/900bd7ac-cdf9-4a2f-8b1f-2c21e3760046/a4783534-f11a-41d1-a455-2e16f5dc258a"
-					(reference "#PWR039")
+					(reference "#PWR044")
 					(unit 1)
 				)
@@
 		(on_board yes)
 		(dnp no)
-		(property "Reference" "#PWR044"
+		(property "Reference" "#PWR049"
 			(at 72.39 114.3 0)
 			(effects
@@
 			(project "SUMEC_MK_IV"
 				(path "/900bd7ac-cdf9-4a2f-8b1f-2c21e3760046/a4783534-f11a-41d1-a455-2e16f5dc258a"
-					(reference "#PWR044")
+					(reference "#PWR049")
 					(unit 1)
 				)
@@
 		(on_board yes)
 		(dnp no)
-		(property "Reference" "#PWR056"
+		(property "Reference" "#PWR061"
 			(at 255.27 114.3 0)
 			(effects
@@
 			(project "SUMEC_MK_IV"
 				(path "/900bd7ac-cdf9-4a2f-8b1f-2c21e3760046/a4783534-f11a-41d1-a455-2e16f5dc258a"
-					(reference "#PWR056")
+					(reference "#PWR061")
 					(unit 1)
 				)
@@
 		(on_board yes)
 		(dnp no)
-		(property "Reference" "#PWR058"
+		(property "Reference" "#PWR063"
 			(at 247.65 111.76 0)
 			(effects
@@
 			(project "SUMEC_MK_IV"
 				(path "/900bd7ac-cdf9-4a2f-8b1f-2c21e3760046/a4783534-f11a-41d1-a455-2e16f5dc258a"
-					(reference "#PWR058")
+					(reference "#PWR063")
 					(unit 1)
 				)
@@
 		(dnp no)
 		(fields_autoplaced yes)
-		(property "Reference" "#PWR045"
+		(property "Reference" "#PWR050"
 			(at 83.82 121.92 0)
 			(effects
@@
 			(project "SUMEC_MK_IV"
 				(path "/900bd7ac-cdf9-4a2f-8b1f-2c21e3760046/a4783534-f11a-41d1-a455-2e16f5dc258a"
-					(reference "#PWR045")
+					(reference "#PWR050")
 					(unit 1)
 				)
@@
 			)
 		)
-		(property "Footprint" ""
+		(property "Footprint" "Connector_Molex:Molex_PicoBlade_53398-0371_1x03-1MP_P1.25mm_Vertical"
 			(at 205.74 104.14 0)
 			(effects
@@
 		(on_board yes)
 		(dnp no)
-		(property "Reference" "#PWR048"
+		(property "Reference" "#PWR053"
 			(at 96.52 161.29 0)
 			(effects
@@
 			(project "SUMEC_MK_IV"
 				(path "/900bd7ac-cdf9-4a2f-8b1f-2c21e3760046/a4783534-f11a-41d1-a455-2e16f5dc258a"
-					(reference "#PWR048")
-					(unit 1)
-				)
+					(reference "#PWR053")
+					(unit 1)
+				)

Commit message: small addition to schematic
Other:
- note added: "I2C signal visualisation? like etherent"
- note added: "qre signal visualisation? (update it on the qre miniboard itself)"
Changed lines of the file:
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@@
+		)
+	)
+	(text "qre signal visualisation? (update it on the qre miniboard itself)"
+		(exclude_from_sim no)
+		(at 180.34 64.77 0)
+		(effects
+			(font
+				(size 1.27 1.27)
+				(color 255 0 0 1)
+			)
 		)
 	)
@@
 		)
 	)
+	(text "I2C signal visualisation? like etherent"
+		(exclude_from_sim no)
+		(at 92.075 101.6 0)
+		(effects
+			(font
+				(size 1.27 1.27)
+				(color 255 0 0 1)
+			)
+		)
+	)

Commit message: PCB routing
Parts:
- U3: footprint sumec-smdV2_library:TSOP -> sumec_brd:TSOP
Changed lines of the file:
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@@
 			)
 		)
-		(property "Footprint" "sumec-smdV2_library:TSOP"
+		(property "Footprint" "sumec_brd:TSOP"
 			(at 83.82 70.485 0)
 			(effects
