File: -PCB-/SUMEC_MK_IV/MCU.kicad_sch (KiCad schematic)
At the start: 25 parts, among them J2 USB_TypeC, SW2 SW_Push, SW3 SW_Push, SW4 SW_Push, SW5 SW_Push, U2 ESP32-S3-WROOM-1, U3 USBLC6-2SC6

Commit message: 3D filepath
Parts:
- removed D3: D_Schottky, Diode_SMD:D_1206_3216Metric_Pad1.42x1.75mm_HandSolder, symbol Device:D_Schottky
Connections:
- net at F1.2: now also J2.A4_B9 (VBUS), J2.B4_A9 (VBUS)
Other:
- note removed: "VBUS Switch already has a Sch Diode solder 1206 0R resistor if not needed"
- moved on the sheet: F1
Changed lines of the file:
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@@
 	(wire
 		(pts
+			(xy 90.17 35.56) (xy 86.36 35.56)
+		)
+		(stroke
+			(width 0)
+			(type default)
+		)
+	)
+	(wire
+		(pts
 			(xy 143.51 132.08) (xy 144.78 132.08)
 		)
@@
 	(wire
 		(pts
+			(xy 97.79 35.56) (xy 101.6 35.56)
+		)
+		(stroke
+			(width 0)
+			(type default)
+		)
+	)
+	(wire
+		(pts
 			(xy 143.51 147.32) (xy 144.78 147.32)
 		)
@@
 		)
 	)
-	(text "VBUS Switch already has a Sch Diode\nsolder 1206 0R resistor if not needed"
-		(exclude_from_sim no)
-		(at 76.2 41.91 0)
-		(effects
-			(font
-				(size 1 1)
-				(color 255 0 0 1)
-			)
-		)
-	)
 	(text "Default Configuration of Strapping Pins\n\nStrapping Pin	Default Configuration		Bit Value\nGPIO0 			Pull-up						1\nGPIO3			Floating						-\nGPIO45			Pull-down					0\nGPIO46			Pull-down					0"
 		(exclude_from_sim no)
@@
 	(symbol
 		(lib_id "Device:Polyfuse")
-		(at 90.17 35.56 90)
+		(at 93.98 35.56 90)
 		(unit 1)
 		(exclude_from_sim no)
@@
 		(dnp no)
 		(property "Reference" "F1"
-			(at 89.535 30.48 90)
+			(at 93.345 30.48 90)
 			(effects
 				(font
@@
 		)
 		(property "Value" "Polyfuse/50R"
-			(at 89.535 32.385 90)
+			(at 93.345 32.385 90)
 			(effects
 				(font
@@
 		)
 		(property "Footprint" "Fuse:Fuse_1206_3216Metric_Pad1.42x1.75mm_HandSolder"
-			(at 95.25 34.29 0)
+			(at 99.06 34.29 0)
 			(effects
 				(font
@@
 		)
 		(property "Datasheet" "~"
-			(at 90.17 35.56 0)
+			(at 93.98 35.56 0)
 			(effects
 				(font
@@
 		)
 		(property "Description" "Resettable fuse, polymeric positive temperature coefficient"
-			(at 90.17 35.56 0)
+			(at 93.98 35.56 0)
 			(effects
 				(font
@@
 					(unit 1)
 				)
-			)
-		)
-	)
-	(symbol
-		(lib_id "Device:D_Schottky")
-		(at 97.79 35.56 0)
-		(unit 1)
-		(exclude_from_sim no)
-		(in_bom yes)
-		(on_board yes)
-		(dnp no)
-		(property "Reference" "D3"
-			(at 99.06 33.02 0)
-			(effects
-				(font
-					(size 1.27 1.27)
-				)
-			)
-		)
-		(property "Value" "D_Schottky"
-			(at 97.79 32.385 0)
-			(effects
-				(font
-					(size 1.27 1.27)
-				)
-				(hide yes)
-			)
-		)
-		(property "Footprint" "Diode_SMD:D_1206_3216Metric_Pad1.42x1.75mm_HandSolder"
-			(at 97.79 35.56 0)
-			(effects
-				(font
-					(size 1.27 1.27)
-				)
-				(hide yes)
-			)
-		)
-		(property "Datasheet" "~"
-			(at 97.79 35.56 0)
-			(effects
-				(font
-					(size 1.27 1.27)
-				)
-				(hide yes)
-			)
-		)
-		(property "Description" "Schottky diode"
-			(at 97.79 35.56 0)
-			(effects
-				(font
-					(size 1.27 1.27)
-				)
-				(hide yes)
-			)
-		)
-		(pin "2"
-		)
-		(pin "1"
-		)
-		(instances
-			(project "SUMEC_MK_IV"
-				(path "/900bd7ac-cdf9-4a2f-8b1f-2c21e3760046/7b93d7c5-db1a-415c-92e4-9ebec6cf195f"
-					(reference "D3")
-					(unit 1)
-				)

Commit message: Some minor changes
BOM update, checked for some pinouts, still some work to do
Parts:
- F1: footprint Fuse:Fuse_1206_3216Metric_Pad1.42x1.75mm_HandSolder -> Fuse:Fuse_0805_2012Metric
Changed lines of the file:
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@@
 	(text "EN=RESET, BOOT=bootloader mode\n\nEnable (EN) is the 3.3V regulator's enable pin. It's\npulled up, so connect to ground to disable the 3.3V\nregulator. This means that you can use this pin\nconnected to a pushbutton to restart your ESP32, for\nexample."
 		(exclude_from_sim no)
-		(at 295.275 132.08 0)
+		(at 293.37 140.335 0)
 		(effects
 			(font
@@
 	(text "Buttons for BOOT and ENABLE functions.\n\nIf the device does not support the auto download mode,\nyou need to get into the download mode manually. \nTo do so, press and hold the BOOT button and then press \nthe RESET button once. After that release the BOOT button."
 		(exclude_from_sim no)
-		(at 295.91 111.125 0)
+		(at 294.005 119.38 0)
 		(effects
 			(font
@@
 			)
 		)
-		(property "Footprint" "Fuse:Fuse_1206_3216Metric_Pad1.42x1.75mm_HandSolder"
+		(property "Footprint" "Fuse:Fuse_0805_2012Metric"
 			(at 99.06 34.29 0)
 			(effects
@@
 			)
 		)
-		(property "Datasheet" "~"
+		(property "Datasheet" "https://cz.mouser.com/ProductDetail/Littelfuse/0805L020-16YR?qs=HoCaDK9Nz5e9OjGjdp4q0Q%3D%3D"
 			(at 93.98 35.56 0)
 			(effects
